File: pcb/senior_project_pcb/io.sch (KiCad schematic (older format))
At the start: 2 parts, among them J1 Conn_01x06, U1 stm32wb55ccu6

Commit message: Add pulse oximeter circuit
Connections:
- no-connect marks 0 -> 28
Changed lines of the file:
@@
 $Descr A4 11693 8268
 encoding utf-8
-Sheet 4 4
+Sheet 4 5
 Title ""
 Date ""
@@
 Text Label 6550 4600 2    50   ~ 0
 JTAG_NTRST
+NoConn ~ 4850 3900
+NoConn ~ 4850 3800
+NoConn ~ 4850 3700
+NoConn ~ 4850 3600
+NoConn ~ 4850 3500
+NoConn ~ 4850 3200
+NoConn ~ 4850 3100
+NoConn ~ 4850 3000
+NoConn ~ 4850 2850
+NoConn ~ 4850 2350
+NoConn ~ 4850 2250
+NoConn ~ 4850 2150
+NoConn ~ 4850 2050
+NoConn ~ 3400 2050
+NoConn ~ 3400 2150
+NoConn ~ 3400 2400
+NoConn ~ 3400 2500
+NoConn ~ 3400 2600
+NoConn ~ 3400 2700
+NoConn ~ 3400 2800
+NoConn ~ 3400 2900
+NoConn ~ 3400 3000
+NoConn ~ 3400 3100
+NoConn ~ 3400 3200
+NoConn ~ 3400 3300
+NoConn ~ 3400 3400
+NoConn ~ 3400 3500
+NoConn ~ 3400 3600
 $EndSCHEMATC

Commit message: Connect up the pulse oximeter and USB
Connections:
- net labels added: SCL, SDA, USB_D+, USB_D-
- wire segments 0 -> 4
- no-connect marks 28 -> 24
Changed lines of the file:
@@
 Text Label 6550 4600 2    50   ~ 0
 JTAG_NTRST
-NoConn ~ 4850 3900
-NoConn ~ 4850 3800
 NoConn ~ 4850 3700
 NoConn ~ 4850 3600
@@
 NoConn ~ 3400 3300
 NoConn ~ 3400 3400
-NoConn ~ 3400 3500
-NoConn ~ 3400 3600
+Text HLabel 5000 3800 2    50   Input ~ 0
+SCL
+Wire Wire Line
+	5000 3800 4850 3800
+Text HLabel 5000 3900 2    50   Input ~ 0
+SDA
+Wire Wire Line
+	5000 3900 4850 3900
+Text HLabel 3150 3600 0    50   Input ~ 0
+USB_D+
+Text HLabel 3150 3500 0    50   Input ~ 0
+USB_D-
+Wire Wire Line
+	3150 3500 3400 3500
+Wire Wire Line
+	3150 3600 3400 3600
 $EndSCHEMATC

Commit message: Add buttons and LEDs
Parts:
- added D2, D3: LED, LED_SMD:LED_0603_1608Metric, symbol Device:LED
- added R10, R11: 330, Resistor_SMD:R_0603_1608Metric, symbol Device:R_Small
- added SW1, SW2: SW_Push_Dual, LL3301NF065QG:LL3301NF065QG, symbol Switch:SW_Push_Dual
Connections:
- net labels added: BTN1, BTN2, LED1, LED2
- no-connect marks 24 -> 22

Commit message: Add temp sensor
Connections:
- net labels added: thermistor, thermopile
- no-connect marks 22 -> 20
Changed lines of the file:
@@
 $Descr A4 11693 8268
 encoding utf-8
-Sheet 4 5
+Sheet 6 6
 Title ""
 Date ""
@@
 JTAG_NTRST
 NoConn ~ 3450 3250
-NoConn ~ 3450 3150
-NoConn ~ 3450 3050
 NoConn ~ 3450 2750
 NoConn ~ 3450 2650
@@
 NoConn ~ 2000 2850
 NoConn ~ 2000 2950
-Text HLabel 3600 3350 2    50   Input ~ 0
+Text HLabel 3600 3350 2    50   BiDi ~ 0
 SCL
 Wire Wire Line
 	3600 3350 3450 3350
-Text HLabel 3600 3450 2    50   Input ~ 0
+Text HLabel 3600 3450 2    50   BiDi ~ 0
 SDA
 Wire Wire Line
 	3600 3450 3450 3450
-Text HLabel 1750 3150 0    50   Input ~ 0
+Text HLabel 1750 3150 0    50   BiDi ~ 0
 USB_D+
-Text HLabel 1750 3050 0    50   Input ~ 0
+Text HLabel 1750 3050 0    50   BiDi ~ 0
 USB_D-
 Wire Wire Line
@@
 Text Label 2000 2250 2    50   ~ 0
 BTN2
+Text HLabel 3450 3050 2    50   Input ~ 0
+thermistor
+Text HLabel 3450 3150 2    50   Input ~ 0
+thermopile
 $EndSCHEMATC

Commit message: Initial layout mostly done
Connections:
- net labels added: INT
- no-connect marks 20 -> 19
Changed lines of the file:
@@
 	0    1    1    0
 $EndComp
+Text Label 3000 4300 2    50   ~ 0
+JTAG_TCK
+Text Label 3000 4400 2    50   ~ 0
+JTAG_TDI
+Text Label 3000 4500 2    50   ~ 0
+JTAG_TDO
 Text Label 3000 4200 2    50   ~ 0
-JTAG_TCK
-Text Label 3000 4300 2    50   ~ 0
-JTAG_TDI
-Text Label 3000 4400 2    50   ~ 0
-JTAG_TDO
-Text Label 3000 4500 2    50   ~ 0
 JTAG_TMS
 Text Label 3000 4600 2    50   ~ 0
@@
 NoConn ~ 2000 1600
 NoConn ~ 2000 1700
-NoConn ~ 2000 2350
-NoConn ~ 2000 2450
-NoConn ~ 2000 2550
 NoConn ~ 2000 2650
 NoConn ~ 2000 2750
@@
 Text Label 5800 2150 0    50   ~ 0
 LED2
-Text Label 2000 1950 2    50   ~ 0
+Text Label 2000 2150 2    50   ~ 0
 LED1
-Text Label 2000 2050 2    50   ~ 0
+Text Label 2000 2250 2    50   ~ 0
 LED2
 $Comp
@@
 NoConn ~ 5350 3500
 NoConn ~ 5350 4150
-Text Label 2000 2150 2    50   ~ 0
+Text Label 2000 2050 2    50   ~ 0
 BTN1
-Text Label 2000 2250 2    50   ~ 0
+Text Label 2000 1950 2    50   ~ 0
 BTN2
-Text HLabel 3450 3050 2    50   Input ~ 0
+Text HLabel 2000 2550 0    50   Input ~ 0
 thermistor
-Text HLabel 3450 3150 2    50   Input ~ 0
+Text HLabel 2000 2450 0    50   Input ~ 0
 thermopile
+Text HLabel 2000 2350 0    50   Input ~ 0
+INT
+NoConn ~ 3450 3150
+NoConn ~ 3450 3050
 $EndSCHEMATC

Commit message: Add ecg sensor
Parts:
- J1: symbol Connector_Generic:Conn_01x06 -> senior_project_pcb-rescue:Conn_01x06-Connector_Generic
- U1: symbol stm32wb55cc:stm32wb55ccu6 -> senior_project_pcb-rescue:stm32wb55ccu6-stm32wb55cc
Changed lines of the file:
@@
 EESchema Schematic File Version 4
-EELAYER 30 0
+LIBS:senior_project_pcb-cache
+EELAYER 29 0
 EELAYER END
 $Descr A4 11693 8268
 encoding utf-8
-Sheet 6 6
+Sheet 6 7
 Title ""
 Date ""
@@
 $EndDescr
 $Comp
-L stm32wb55cc:stm32wb55ccu6 U?
+L senior_project_pcb-rescue:stm32wb55ccu6-stm32wb55cc U?
 U 1 1 5FC33073
 P 2700 2150
@@
 JTAG_NTRST
 $Comp
-L Connector_Generic:Conn_01x06 J1
+L senior_project_pcb-rescue:Conn_01x06-Connector_Generic J1
 U 1 1 5FC38CA8
 P 3200 4300

Commit message: Add RF/Bluetooth to PCB
Parts:
- removed J1: Conn_01x06, Connector_PinHeader_2.54mm:PinHeader_1x06_P2.54mm_Vertical, symbol senior_project_pcb-rescue:Conn_01x06-Connector_Generic
- added J1: Conn_02x03_Odd_Even, Connector_PinHeader_2.54mm:PinHeader_2x03_P2.54mm_Vertical, symbol Connector_Generic:Conn_02x03_Odd_Even
- added Y1: Crystal_GND24, Crystal:Crystal_SMD_2016-4Pin_2.0x1.6mm, symbol Device:Crystal_GND24
- U1: symbol senior_project_pcb-rescue:stm32wb55ccu6-stm32wb55cc -> senior_project_pcb-rescue:stm32wb55ccu6-stm32wb55cc-senior_project_pcb-rescue
Connections:
- net GND: now also J1.6 (Pin_6), Y1.2, Y1.4
- net JTAG_NTRST: now also J1.5 (Pin_5)
- net JTAG_TCK: now also J1.2 (Pin_2)
- net JTAG_TDI: now also J1.3 (Pin_3)
- net JTAG_TDO: now also J1.4 (Pin_4)
- net JTAG_TMS: now also J1.1 (Pin_1)
- net thermistor: now also U1.17 (PA8); no longer U1.15 (PA6)
- net thermopile: now also U1.16 (PA7); no longer U1.14 (PA5)
- net at U1.24 (OSC_OUT): now also Y1.1
- net at U1.25 (OSC_IN): now also Y1.3
- new net ECG_OUT: U1.15 (PA6)
- new net ECG_SDN: U1.14 (PA5)
- no-connect marks 19 -> 15

Commit message: PCB Update
Parts:
- D2, D3: Manufacturer_Name (none) -> Wurth Elektronik; Manufacturer_Part_Number (none) -> 150060RS75000; Mouser Part Number (none) -> 710-150060RS75000
- R10, R11: Manufacturer_Name (none) -> Yageo; Manufacturer_Part_Number (none) -> RC0603JR-07330RL; Mouser Part Number (none) -> 603-RC0603JR-07330RL
- SW1, SW2: Manufacturer_Name (none) -> E-Switch; Manufacturer_Part_Number (none) -> LL3301NF065QG; Mouser Part Number (none) -> 612-LL3301NF065QG
- U1: Manufacturer_Name (none) -> STMicro; Manufacturer_Part_Number (none) -> STM32WB55CEU6; Mouser Part Number (none) -> 511-STM32WB55CEU6
- Y1: Manufacturer_Name (none) -> Murata; Manufacturer_Part_Number (none) -> XRCGB32M000F2P02R0; Mouser Part Number (none) -> 81-XRCGB32M000F2P02R
Connections:
- net BTN1: now also U1.46 (PB6); no longer U1.10 (PA1)
- net BTN2: now also U1.47 (PB7); no longer U1.9 (PA0)
- net LO+: now reaches U1.18 (PA9)
- net LO-: now reaches U1.19 (PB2)
- no-connect marks 15 -> 13
Changed lines of the file:
@@
 Text Label 2600 5150 2    50   ~ 0
 JTAG_NTRST
-NoConn ~ 3450 3250
-NoConn ~ 3450 2750
 NoConn ~ 3450 2650
 NoConn ~ 3450 2550
@@
 NoConn ~ 2000 1600
 NoConn ~ 2000 1700
-NoConn ~ 2000 2850
-NoConn ~ 2000 2950
 Text HLabel 3600 3350 2    50   BiDi ~ 0
 SCL
@@
 F 2 "LED_SMD:LED_0603_1608Metric" H 5400 2500 50  0001 C CNN
 F 3 "~" H 5400 2500 50  0001 C CNN
+F 4 "Wurth Elektronik" H 5400 2500 50  0001 C CNN "Manufacturer_Name"
+F 5 "150060RS75000" H 5400 2500 50  0001 C CNN "Manufacturer_Part_Number"
+F 6 "710-150060RS75000" H 5400 2500 50  0001 C CNN "Mouser Part Number"
 	1    5400 2500
 	0    -1   -1   0
@@
 F 2 "LED_SMD:LED_0603_1608Metric" H 5800 2500 50  0001 C CNN
 F 3 "~" H 5800 2500 50  0001 C CNN
+F 4 "Wurth Elektronik" H 5800 2500 50  0001 C CNN "Manufacturer_Name"
+F 5 "150060RS75000" H 5800 2500 50  0001 C CNN "Manufacturer_Part_Number"
+F 6 "710-150060RS75000" H 5800 2500 50  0001 C CNN "Mouser Part Number"
 	1    5800 2500
 	0    -1   -1   0
@@
 F 2 "Resistor_SMD:R_0603_1608Metric" H 5800 2250 50  0001 C CNN
 F 3 "~" H 5800 2250 50  0001 C CNN
+F 4 "Yageo" H 5800 2250 50  0001 C CNN "Manufacturer_Name"
+F 5 "RC0603JR-07330RL" H 5800 2250 50  0001 C CNN "Manufacturer_Part_Number"
+F 6 " 603-RC0603JR-07330RL " H 5800 2250 50  0001 C CNN "Mouser Part Number"
 	1    5800 2250
 	1    0    0    -1
@@
 F 2 "Resistor_SMD:R_0603_1608Metric" H 5400 2250 50  0001 C CNN
 F 3 "~" H 5400 2250 50  0001 C CNN
+F 4 "Yageo" H 5400 2250 50  0001 C CNN "Manufacturer_Name"
+F 5 "RC0603JR-07330RL" H 5400 2250 50  0001 C CNN "Manufacturer_Part_Number"
+F 6 " 603-RC0603JR-07330RL " H 5400 2250 50  0001 C CNN "Mouser Part Number"
 	1    5400 2250
 	1    0    0    -1
@@
 F 2 "LL3301NF065QG:LL3301NF065QG" H 5550 3700 50  0001 C CNN
 F 3 "~" H 5550 3700 50  0001 C CNN
+F 4 "E-Switch" H 5550 3500 50  0001 C CNN "Manufacturer_Name"
+F 5 "LL3301NF065QG " H 5550 3500 50  0001 C CNN "Manufacturer_Part_Number"
+F 6 " 612-LL3301NF065QG " H 5550 3500 50  0001 C CNN "Mouser Part Number"
 	1    5550 3500
 	1    0    0    -1
@@
 F 2 "LL3301NF065QG:LL3301NF065QG" H 5550 4350 50  0001 C CNN
 F 3 "~" H 5550 4350 50  0001 C CNN
+F 4 "E-Switch" H 5550 4150 50  0001 C CNN "Manufacturer_Name"
+F 5 "LL3301NF065QG " H 5550 4150 50  0001 C CNN "Manufacturer_Part_Number"
+F 6 " 612-LL3301NF065QG " H 5550 4150 50  0001 C CNN "Mouser Part Number"
 	1    5550 4150
 	1    0    0    -1
@@
 NoConn ~ 5350 3500
 NoConn ~ 5350 4150
-Text Label 2000 2050 2    50   ~ 0
+Text Label 3450 3150 0    50   ~ 0
 BTN1
-Text Label 2000 1950 2    50   ~ 0
+Text Label 3450 3250 0    50   ~ 0
 BTN2
-Text HLabel 2000 2750 0    50   Input ~ 0
-thermistor
-Text HLabel 2000 2650 0    50   Input ~ 0
-thermopile
 Text HLabel 2000 2350 0    50   Input ~ 0
 INT
-NoConn ~ 3450 3150
 NoConn ~ 3450 3050
-Text HLabel 2000 2550 0    50   Input ~ 0
-ECG_OUT
-Text HLabel 2000 2450 0    50   Input ~ 0
-ECG_SDN
 $Comp
 L Device:Crystal_GND24 Y1
@@
 F 2 "Crystal:Crystal_SMD_2016-4Pin_2.0x1.6mm" H 3950 1800 50  0001 C CNN
 F 3 "~" H 3950 1800 50  0001 C CNN
+F 4 "Murata" H 3950 1800 50  0001 C CNN "Manufacturer_Name"
+F 5 "XRCGB32M000F2P02R0" H 3950 1800 50  0001 C CNN "Manufacturer_Part_Number"
+F 6 " 81-XRCGB32M000F2P02R " H 3950 1800 50  0001 C CNN "Mouser Part Number"
 	1    3950 1800
+	1    0    0    -1
+$EndComp
+Wire Wire Line
+	3450 1800 3800 1800
+Wire Wire Line
+	3450 1900 3450 2100
+Wire Wire Line
+	3450 2100 4100 2100
+Wire Wire Line
+	4100 2100 4100 1800
+$Comp
+L power:GND #PWR0109
+U 1 1 60320491
+P 3950 2000
+F 0 "#PWR0109" H 3950 1750 50  0001 C CNN
+F 1 "GND" H 3955 1827 50  0000 C CNN
+F 2 "" H 3950 2000 50  0001 C CNN
+F 3 "" H 3950 2000 50  0001 C CNN
+	1    3950 2000
+	1    0    0    -1
+$EndComp
+$Comp
+L power:GND #PWR0118
+U 1 1 6032099A
+P 3950 1600
+F 0 "#PWR0118" H 3950 1350 50  0001 C CNN
+F 1 "GND" H 3955 1427 50  0000 C CNN
+F 2 "" H 3950 1600 50  0001 C CNN
+F 3 "" H 3950 1600 50  0001 C CNN
+	1    3950 1600
+	-1   0    0    1
+$EndComp
+$Comp
+L Connector_Generic:Conn_02x03_Odd_Even J1
+U 1 1 60340AB4
+P 2800 5050
+F 0 "J1" H 2850 5367 50  0000 C CNN
+F 1 "Conn_02x03_Odd_Even" H 2850 5276 50  0000 C CNN
+F 2 "Connector_PinHeader_2.54mm:PinHeader_2x03_P2.54mm_Vertical" H 2800 5050 50  0001 C CNN
+F 3 "~" H 2800 5050 50  0001 C CNN
+	1    2800 5050
 	1    0    0    -1
 $EndComp
@@
 F 2 "Package_DFN_QFN:QFN-48-1EP_7x7mm_P0.5mm_EP5.6x5.6mm" H 2750 2850 50  0001 C CNN
 F 3 "" H 2750 2850 50  0001 C CNN
+F 4 "STMicro" H 2700 2150 50  0001 C CNN "Manufacturer_Name"
+F 5 "STM32WB55CEU6" H 2700 2150 50  0001 C CNN "Manufacturer_Part_Number"
+F 6 "511-STM32WB55CEU6" H 2700 2150 50  0001 C CNN "Mouser Part Number"
 	1    2700 2150
 	1    0    0    -1
 $EndComp
-Wire Wire Line
-	3450 1800 3800 1800
-Wire Wire Line
-	3450 1900 3450 2100
-Wire Wire Line
-	3450 2100 4100 2100
-Wire Wire Line
-	4100 2100 4100 1800
-$Comp
-L power:GND #PWR0109
-U 1 1 60320491
-P 3950 2000
-F 0 "#PWR0109" H 3950 1750 50  0001 C CNN
-F 1 "GND" H 3955 1827 50  0000 C CNN
-F 2 "" H 3950 2000 50  0001 C CNN
-F 3 "" H 3950 2000 50  0001 C CNN
-	1    3950 2000
-	1    0    0    -1
-$EndComp
-$Comp
-L power:GND #PWR0118
-U 1 1 6032099A
-P 3950 1600
-F 0 "#PWR0118" H 3950 1350 50  0001 C CNN
-F 1 "GND" H 3955 1427 50  0000 C CNN
-F 2 "" H 3950 1600 50  0001 C CNN
-F 3 "" H 3950 1600 50  0001 C CNN
-	1    3950 1600
-	-1   0    0    1
-$EndComp
-$Comp
-L Connector_Generic:Conn_02x03_Odd_Even J1
-U 1 1 60340AB4
-P 2800 5050
-F 0 "J1" H 2850 5367 50  0000 C CNN
-F 1 "Conn_02x03_Odd_Even" H 2850 5276 50  0000 C CNN
-F 2 "Connector_PinHeader_2.54mm:PinHeader_2x03_P2.54mm_Vertical" H 2800 5050 50  0001 C CNN
-F 3 "~" H 2800 5050 50  0001 C CNN
-	1    2800 5050
-	1    0    0    -1
-$EndComp
+Text HLabel 2000 2450 0    50   Input ~ 0
+ECG_SDN
+Text HLabel 2000 2550 0    50   Input ~ 0
+ECG_OUT
+Text HLabel 2000 2650 0    50   Input ~ 0
+thermopile
+Text HLabel 2000 2750 0    50   Input ~ 0
+thermistor
+Text HLabel 2000 2850 0    50   Input ~ 0
+LO+
+Text HLabel 3450 2750 2    50   Input ~ 0
+LO-
+NoConn ~ 2000 2950
+NoConn ~ 2000 1950
+NoConn ~ 2000 2050
 $EndSCHEMATC
