File: pcb/senior_project_pcb/io.sch (KiCad schematic (older format))
At the start: 9 parts, among them J1 Conn_02x03_Odd_Even, SW1 SW_Push_Dual, SW2 SW_Push_Dual, U1 stm32wb55ccu6, Y1 Crystal_GND24

Commit message: Send PCB off for manufacture
Parts:
- J1: Manufacturer_Name (none) -> Molex; Manufacturer_Part_Number (none) -> 10-89-7061; Mouser Part Number (none) -> 538-10-89-7061
Changed lines of the file:
@@
 F 2 "Connector_PinHeader_2.54mm:PinHeader_2x03_P2.54mm_Vertical" H 2800 5050 50  0001 C CNN
 F 3 "~" H 2800 5050 50  0001 C CNN
+F 4 "Molex" H 2800 5050 50  0001 C CNN "Manufacturer_Name"
+F 5 "10-89-7061" H 2800 5050 50  0001 C CNN "Manufacturer_Part_Number"
+F 6 "538-10-89-7061" H 2800 5050 50  0001 C CNN "Mouser Part Number"
 	1    2800 5050
 	1    0    0    -1
