File: pcb/senior_project_pcb/ecg.sch (KiCad schematic (older format))
At the start: 24 parts, among them J4 Conn_01x03, U2 AD8232ACPZ-R7

Commit message: PCB Update
Parts:
- C15: Manufacturer_Name (none) -> AVX; Manufacturer_Part_Number (none) -> 06035D103KAT2A; Mouser Part Number (none) -> 581-06035D103KAT2A
- C16: value .33uF -> .33u; Manufacturer_Name (none) -> Kamaya; Manufacturer_Part_Number (none) -> 0603X334J160CT; Mouser Part Number (none) -> 791-0603X334J160CT
- C17: Manufacturer_Name (none) -> Kamaya; Manufacturer_Part_Number (none) -> 0603X334J160CT; Mouser Part Number (none) -> 791-0603X334J160CT
- C6: Manufacturer_Name (none) -> Walsin; Manufacturer_Part_Number (none) -> 0603N152J250CT; Mouser Part Number (none) -> 791-0603N152J250CT
- C7: Manufacturer_Name (none) -> AVX; Manufacturer_Part_Number (none) -> 06035A102JAT2A; Mouser Part Number (none) -> 581-06035A102J
- R17: Manufacturer_Name (none) -> Yageo; Manufacturer_Part_Number (none) -> RC0603FR-07360KL; Mouser Part Number (none) -> 603-RC0603FR-07360KL
- R18, R19: Manufacturer_Name (none) -> Yageo; Manufacturer_Part_Number (none) -> RC0603FR-10180KL; Mouser Part Number (none) -> 603-RC0603FR-10180KL
- R20, R22, R23: Manufacturer_Name (none) -> Yageo; Manufacturer_Part_Number (none) -> RC0603FR-071ML; Mouser Part Number (none) -> 603-RC0603FR-071ML
- R24, R25, R27, R28, R8, R9: Manufacturer_Name (none) -> Vishay; Manufacturer_Part_Number (none) -> CRCW060310M0FKEAC; Mouser Part Number (none) -> 71-CRCW060310M0FKEAC
- R26: Manufacturer_Name (none) -> Yageo; Manufacturer_Part_Number (none) -> RC0603FR-071M4L; Mouser Part Number (none) -> 603-RC0603FR-071M4L
- U2: Manufacturer_Name (none) -> Analog; Manufacturer_Part_Number (none) -> AD8232ACPZ-R7; Mouser Part Number (none) -> 584-AD8232ACPZ-R7
Connections:
- net LO-: now reaches U2.11 (LOD-)
- net LO+: now reaches U2.12 (LOD+)
- no-connect marks 2 -> 0
Changed lines of the file:
@@
 F 2 "Package_CSP:LFCSP-20-1EP_4x4mm_P0.5mm_EP2.1x2.1mm" H 5550 4040 60  0001 C CNN
 F 3 "" H 4150 3800 60  0000 C CNN
+F 4 "Analog" H 4150 3800 50  0001 C CNN "Manufacturer_Name"
+F 5 "AD8232ACPZ-R7" H 4150 3800 50  0001 C CNN "Manufacturer_Part_Number"
+F 6 "584-AD8232ACPZ-R7" H 4150 3800 50  0001 C CNN "Mouser Part Number"
 	1    4150 3800
 	1    0    0    -1
@@
 P 4900 3300
 F 0 "C16" V 4648 3300 50  0000 C CNN
-F 1 ".33uF" V 4739 3300 50  0000 C CNN
+F 1 ".33u" V 4739 3300 50  0000 C CNN
 F 2 "Capacitor_SMD:C_0603_1608Metric" H 4938 3150 50  0001 C CNN
 F 3 "~" H 4900 3300 50  0001 C CNN
+F 4 "Kamaya" H 4900 3300 50  0001 C CNN "Manufacturer_Name"
+F 5 "0603X334J160CT" H 4900 3300 50  0001 C CNN "Manufacturer_Part_Number"
+F 6 "791-0603X334J160CT" H 4900 3300 50  0001 C CNN "Mouser Part Number"
 	1    4900 3300
 	0    1    1    0
@@
 F 2 "Resistor_SMD:R_0603_1608Metric" H 3450 3900 50  0001 C CNN
 F 3 "~" H 3450 3900 50  0001 C CNN
+F 4 "Yageo" H 3450 3900 50  0001 C CNN "Manufacturer_Name"
+F 5 "RC0603FR-10180KL" H 3450 3900 50  0001 C CNN "Manufacturer_Part_Number"
+F 6 " 603-RC0603FR-10180KL " H 3450 3900 50  0001 C CNN "Mouser Part Number"
 	1    3450 3900
 	0    1    1    0
@@
 F 2 "Resistor_SMD:R_0603_1608Metric" H 3450 4000 50  0001 C CNN
 F 3 "~" H 3450 4000 50  0001 C CNN
+F 4 "Yageo" H 3450 4000 50  0001 C CNN "Manufacturer_Name"
+F 5 "RC0603FR-10180KL" H 3450 4000 50  0001 C CNN "Manufacturer_Part_Number"
+F 6 " 603-RC0603FR-10180KL " H 3450 4000 50  0001 C CNN "Mouser Part Number"
 	1    3450 4000
 	0    1    1    0
@@
 F 2 "Resistor_SMD:R_0603_1608Metric" H 2900 3650 50  0001 C CNN
 F 3 "~" H 2900 3650 50  0001 C CNN
+F 4 "Vishay" H 2900 3650 50  0001 C CNN "Manufacturer_Name"
+F 5 "CRCW060310M0FKEAC" H 2900 3650 50  0001 C CNN "Manufacturer_Part_Number"
+F 6 " 71-CRCW060310M0FKEAC " H 2900 3650 50  0001 C CNN "Mouser Part Number"
 	1    2900 3650
 	-1   0    0    1
@@
 F 2 "Resistor_SMD:R_0603_1608Metric" H 2700 3750 50  0001 C CNN
 F 3 "~" H 2700 3750 50  0001 C CNN
+F 4 "Vishay" H 2700 3750 50  0001 C CNN "Manufacturer_Name"
+F 5 "CRCW060310M0FKEAC" H 2700 3750 50  0001 C CNN "Manufacturer_Part_Number"
+F 6 " 71-CRCW060310M0FKEAC " H 2700 3750 50  0001 C CNN "Mouser Part Number"
 	1    2700 3750
 	-1   0    0    1
@@
 F 2 "Capacitor_SMD:C_0603_1608Metric" H 4000 4400 50  0001 C CNN
 F 3 "~" H 4000 4400 50  0001 C CNN
+F 4 "AVX" H 4000 4400 50  0001 C CNN "Manufacturer_Name"
+F 5 "06035A102JAT2A" H 4000 4400 50  0001 C CNN "Manufacturer_Part_Number"
+F 6 " 581-06035A102J " H 4000 4400 50  0001 C CNN "Mouser Part Number"
 	1    4000 4400
 	1    0    0    -1
@@
 F 2 "Resistor_SMD:R_0603_1608Metric" H 3300 4500 50  0001 C CNN
 F 3 "~" H 3300 4500 50  0001 C CNN
+F 4 "Yageo" H 3300 4500 50  0001 C CNN "Manufacturer_Name"
+F 5 "RC0603FR-07360KL" H 3300 4500 50  0001 C CNN "Manufacturer_Part_Number"
+F 6 " 603-RC0603FR-07360KL " H 3300 4500 50  0001 C CNN "Mouser Part Number"
 	1    3300 4500
 	0    1    1    0
@@
 F 2 "Resistor_SMD:R_0603_1608Metric" H 6000 3800 50  0001 C CNN
 F 3 "~" H 6000 3800 50  0001 C CNN
+F 4 "Vishay" H 6000 3800 50  0001 C CNN "Manufacturer_Name"
+F 5 "CRCW060310M0FKEAC" H 6000 3800 50  0001 C CNN "Manufacturer_Part_Number"
+F 6 " 71-CRCW060310M0FKEAC " H 6000 3800 50  0001 C CNN "Mouser Part Number"
 	1    6000 3800
 	0    1    1    0
@@
 F 2 "Resistor_SMD:R_0603_1608Metric" H 6250 3700 50  0001 C CNN
 F 3 "~" H 6250 3700 50  0001 C CNN
+F 4 "Yageo" H 6250 3700 50  0001 C CNN "Manufacturer_Name"
+F 5 "RC0603FR-071M4L" H 6250 3700 50  0001 C CNN "Manufacturer_Part_Number"
+F 6 " 603-RC0603FR-071M4L " H 6250 3700 50  0001 C CNN "Mouser Part Number"
 	1    6250 3700
 	-1   0    0    1
@@
 F 2 "Resistor_SMD:R_0603_1608Metric" H 6250 3900 50  0001 C CNN
 F 3 "~" H 6250 3900 50  0001 C CNN
+F 4 "Vishay" H 6250 3900 50  0001 C CNN "Manufacturer_Name"
+F 5 "CRCW060310M0FKEAC" H 6250 3900 50  0001 C CNN "Manufacturer_Part_Number"
+F 6 " 71-CRCW060310M0FKEAC " H 6250 3900 50  0001 C CNN "Mouser Part Number"
 	1    6250 3900
 	-1   0    0    1
@@
 F 2 "Capacitor_SMD:C_0603_1608Metric" H 6450 3600 50  0001 C CNN
 F 3 "~" H 6450 3600 50  0001 C CNN
+F 4 "Kamaya" H 6450 3600 50  0001 C CNN "Manufacturer_Name"
+F 5 "0603X334J160CT" H 6450 3600 50  0001 C CNN "Manufacturer_Part_Number"
+F 6 "791-0603X334J160CT" H 6450 3600 50  0001 C CNN "Mouser Part Number"
 	1    6450 3600
 	0    -1   -1   0
@@
 F 2 "Resistor_SMD:R_0603_1608Metric" H 3800 4900 50  0001 C CNN
 F 3 "~" H 3800 4900 50  0001 C CNN
+F 4 "Yageo" H 3800 4900 50  0001 C CNN "Manufacturer_Name"
+F 5 "RC0603FR-071ML" H 3800 4900 50  0001 C CNN "Manufacturer_Part_Number"
+F 6 " 603-RC0603FR-071ML " H 3800 4900 50  0001 C CNN "Mouser Part Number"
 	1    3800 4900
 	0    1    1    0
@@
 F 2 "Capacitor_SMD:C_0603_1608Metric" H 4050 5000 50  0001 C CNN
 F 3 "~" H 4050 5000 50  0001 C CNN
+F 4 "AVX" H 4050 5000 50  0001 C CNN "Manufacturer_Name"
+F 5 "06035D103KAT2A" H 4050 5000 50  0001 C CNN "Manufacturer_Part_Number"
+F 6 "581-06035D103KAT2A" H 4050 5000 50  0001 C CNN "Mouser Part Number"
 	1    4050 5000
 	1    0    0    -1
@@
 F 2 "Resistor_SMD:R_0603_1608Metric" H 3550 4800 50  0001 C CNN
 F 3 "~" H 3550 4800 50  0001 C CNN
+F 4 "Yageo" H 3550 4800 50  0001 C CNN "Manufacturer_Name"
+F 5 "RC0603FR-071ML" H 3550 4800 50  0001 C CNN "Manufacturer_Part_Number"
+F 6 " 603-RC0603FR-071ML " H 3550 4800 50  0001 C CNN "Mouser Part Number"
 	1    3550 4800
 	-1   0    0    1
@@
 F 2 "Resistor_SMD:R_0603_1608Metric" H 3750 5400 50  0001 C CNN
 F 3 "~" H 3750 5400 50  0001 C CNN
+F 4 "Yageo" H 3750 5400 50  0001 C CNN "Manufacturer_Name"
+F 5 "RC0603FR-071ML" H 3750 5400 50  0001 C CNN "Manufacturer_Part_Number"
+F 6 " 603-RC0603FR-071ML " H 3750 5400 50  0001 C CNN "Mouser Part Number"
 	1    3750 5400
 	1    0    0    -1
@@
 F 2 "Capacitor_SMD:C_0603_1608Metric" H 3550 5400 50  0001 C CNN
 F 3 "~" H 3550 5400 50  0001 C CNN
+F 4 "Walsin" H 3550 5400 50  0001 C CNN "Manufacturer_Name"
+F 5 "0603N152J250CT" H 3550 5400 50  0001 C CNN "Manufacturer_Part_Number"
+F 6 "791-0603N152J250CT" H 3550 5400 50  0001 C CNN "Mouser Part Number"
 	1    3550 5400
 	1    0    0    -1
@@
 F 2 "Resistor_SMD:R_0603_1608Metric" H 5900 4400 50  0001 C CNN
 F 3 "~" H 5900 4400 50  0001 C CNN
+F 4 "Vishay" H 5900 4400 50  0001 C CNN "Manufacturer_Name"
+F 5 "CRCW060310M0FKEAC" H 5900 4400 50  0001 C CNN "Manufacturer_Part_Number"
+F 6 " 71-CRCW060310M0FKEAC " H 5900 4400 50  0001 C CNN "Mouser Part Number"
 	1    5900 4400
 	-1   0    0    1
@@
 F 2 "Resistor_SMD:R_0603_1608Metric" H 6400 4400 50  0001 C CNN
 F 3 "~" H 6400 4400 50  0001 C CNN
+F 4 "Vishay" H 6400 4400 50  0001 C CNN "Manufacturer_Name"
+F 5 "CRCW060310M0FKEAC" H 6400 4400 50  0001 C CNN "Manufacturer_Part_Number"
+F 6 " 71-CRCW060310M0FKEAC " H 6400 4400 50  0001 C CNN "Mouser Part Number"
 	1    6400 4400
 	-1   0    0    1
@@
 Text HLabel 5750 5300 2    50   Input ~ 0
 ECG_SDN
-NoConn ~ 5750 5400
-NoConn ~ 5750 5500
 Wire Wire Line
 	3550 2800 3550 4700
@@
 Text Label 2000 4700 0    50   ~ 0
 REFOUT
+Text HLabel 5750 5400 2    50   Output ~ 0
+LO+
+Text HLabel 5750 5500 2    50   Output ~ 0
+LO-
 $EndSCHEMATC

Commit message: Send PCB off for manufacture
Parts:
- C16, C17: Manufacturer_Name Kamaya -> Samsung; Manufacturer_Part_Number 0603X334J160CT -> CL10B334KO8NNNC; Mouser Part Number 791-0603X334J160CT -> 187-CL10B334KO8NNNC
- C20, C21: Manufacturer_Name (none) -> AVX; Manufacturer_Part_Number (none) -> 0603YC104MAT4A; Mouser Part Number (none) -> 581-0603YC104MAT4A
- R21: Manufacturer_Name (none) -> Yageo; Manufacturer_Part_Number (none) -> RC0603FR-13100KL; Mouser Part Number (none) -> 603-RC0603FR-13100KL
- R24, R25, R27, R28, R8, R9: Manufacturer_Name Vishay -> Yageo; Manufacturer_Part_Number CRCW060310M0FKEAC -> RC0603FR-1010ML; Mouser Part Number 71-CRCW060310M0FKEAC -> 603-RC0603FR-1010ML
Changed lines of the file:
@@
 F 2 "Capacitor_SMD:C_0603_1608Metric" H 4938 3150 50  0001 C CNN
 F 3 "~" H 4900 3300 50  0001 C CNN
-F 4 "Kamaya" H 4900 3300 50  0001 C CNN "Manufacturer_Name"
-F 5 "0603X334J160CT" H 4900 3300 50  0001 C CNN "Manufacturer_Part_Number"
-F 6 "791-0603X334J160CT" H 4900 3300 50  0001 C CNN "Mouser Part Number"
+F 4 "Samsung" H 4900 3300 50  0001 C CNN "Manufacturer_Name"
+F 5 "CL10B334KO8NNNC" H 4900 3300 50  0001 C CNN "Manufacturer_Part_Number"
+F 6 "187-CL10B334KO8NNNC" H 4900 3300 50  0001 C CNN "Mouser Part Number"
 	1    4900 3300
 	0    1    1    0
@@
 F 2 "Resistor_SMD:R_0603_1608Metric" H 2900 3650 50  0001 C CNN
 F 3 "~" H 2900 3650 50  0001 C CNN
-F 4 "Vishay" H 2900 3650 50  0001 C CNN "Manufacturer_Name"
-F 5 "CRCW060310M0FKEAC" H 2900 3650 50  0001 C CNN "Manufacturer_Part_Number"
-F 6 " 71-CRCW060310M0FKEAC " H 2900 3650 50  0001 C CNN "Mouser Part Number"
+F 4 "Yageo" H 2900 3650 50  0001 C CNN "Manufacturer_Name"
+F 5 "RC0603FR-1010ML" H 2900 3650 50  0001 C CNN "Manufacturer_Part_Number"
+F 6 " 603-RC0603FR-1010ML " H 2900 3650 50  0001 C CNN "Mouser Part Number"
 	1    2900 3650
 	-1   0    0    1
@@
 F 2 "Resistor_SMD:R_0603_1608Metric" H 2700 3750 50  0001 C CNN
 F 3 "~" H 2700 3750 50  0001 C CNN
-F 4 "Vishay" H 2700 3750 50  0001 C CNN "Manufacturer_Name"
-F 5 "CRCW060310M0FKEAC" H 2700 3750 50  0001 C CNN "Manufacturer_Part_Number"
-F 6 " 71-CRCW060310M0FKEAC " H 2700 3750 50  0001 C CNN "Mouser Part Number"
+F 4 "Yageo" H 2700 3750 50  0001 C CNN "Manufacturer_Name"
+F 5 "RC0603FR-1010ML" H 2700 3750 50  0001 C CNN "Manufacturer_Part_Number"
+F 6 " 603-RC0603FR-1010ML " H 2700 3750 50  0001 C CNN "Mouser Part Number"
 	1    2700 3750
 	-1   0    0    1
@@
 F 2 "Resistor_SMD:R_0603_1608Metric" H 6000 3800 50  0001 C CNN
 F 3 "~" H 6000 3800 50  0001 C CNN
-F 4 "Vishay" H 6000 3800 50  0001 C CNN "Manufacturer_Name"
-F 5 "CRCW060310M0FKEAC" H 6000 3800 50  0001 C CNN "Manufacturer_Part_Number"
-F 6 " 71-CRCW060310M0FKEAC " H 6000 3800 50  0001 C CNN "Mouser Part Number"
+F 4 "Yageo" H 6000 3800 50  0001 C CNN "Manufacturer_Name"
+F 5 "RC0603FR-1010ML" H 6000 3800 50  0001 C CNN "Manufacturer_Part_Number"
+F 6 " 603-RC0603FR-1010ML " H 6000 3800 50  0001 C CNN "Mouser Part Number"
 	1    6000 3800
 	0    1    1    0
@@
 F 2 "Resistor_SMD:R_0603_1608Metric" H 6250 3900 50  0001 C CNN
 F 3 "~" H 6250 3900 50  0001 C CNN
-F 4 "Vishay" H 6250 3900 50  0001 C CNN "Manufacturer_Name"
-F 5 "CRCW060310M0FKEAC" H 6250 3900 50  0001 C CNN "Manufacturer_Part_Number"
-F 6 " 71-CRCW060310M0FKEAC " H 6250 3900 50  0001 C CNN "Mouser Part Number"
+F 4 "Yageo" H 6250 3900 50  0001 C CNN "Manufacturer_Name"
+F 5 "RC0603FR-1010ML" H 6250 3900 50  0001 C CNN "Manufacturer_Part_Number"
+F 6 " 603-RC0603FR-1010ML " H 6250 3900 50  0001 C CNN "Mouser Part Number"
 	1    6250 3900
 	-1   0    0    1
@@
 F 2 "Capacitor_SMD:C_0603_1608Metric" H 6450 3600 50  0001 C CNN
 F 3 "~" H 6450 3600 50  0001 C CNN
-F 4 "Kamaya" H 6450 3600 50  0001 C CNN "Manufacturer_Name"
-F 5 "0603X334J160CT" H 6450 3600 50  0001 C CNN "Manufacturer_Part_Number"
-F 6 "791-0603X334J160CT" H 6450 3600 50  0001 C CNN "Mouser Part Number"
+F 4 "Samsung" H 6450 3600 50  0001 C CNN "Manufacturer_Name"
+F 5 "CL10B334KO8NNNC" H 6450 3600 50  0001 C CNN "Manufacturer_Part_Number"
+F 6 "187-CL10B334KO8NNNC" H 6450 3600 50  0001 C CNN "Mouser Part Number"
 	1    6450 3600
 	0    -1   -1   0
@@
 F 2 "Resistor_SMD:R_0603_1608Metric" H 3750 5200 50  0001 C CNN
 F 3 "~" H 3750 5200 50  0001 C CNN
+F 4 "Yageo" H 3750 5200 50  0001 C CNN "Manufacturer_Name"
+F 5 "RC0603FR-13100KL" H 3750 5200 50  0001 C CNN "Manufacturer_Part_Number"
+F 6 " 603-RC0603FR-13100KL " H 3750 5200 50  0001 C CNN "Mouser Part Number"
 	1    3750 5200
 	1    0    0    -1
@@
 F 2 "Capacitor_SMD:C_0603_1608Metric" H 7350 4650 50  0001 C CNN
 F 3 "~" H 7350 4650 50  0001 C CNN
+F 4 "AVX" H 7350 4650 50  0001 C CNN "Manufacturer_Name"
+F 5 "0603YC104MAT4A" H 7350 4650 50  0001 C CNN "Manufacturer_Part_Number"
+F 6 "581-0603YC104MAT4A" H 7350 4650 50  0001 C CNN "Mouser Part Number"
 	1    7350 4650
 	1    0    0    -1
@@
 F 2 "Resistor_SMD:R_0603_1608Metric" H 5900 4400 50  0001 C CNN
 F 3 "~" H 5900 4400 50  0001 C CNN
-F 4 "Vishay" H 5900 4400 50  0001 C CNN "Manufacturer_Name"
-F 5 "CRCW060310M0FKEAC" H 5900 4400 50  0001 C CNN "Manufacturer_Part_Number"
-F 6 " 71-CRCW060310M0FKEAC " H 5900 4400 50  0001 C CNN "Mouser Part Number"
+F 4 "Yageo" H 5900 4400 50  0001 C CNN "Manufacturer_Name"
+F 5 "RC0603FR-1010ML" H 5900 4400 50  0001 C CNN "Manufacturer_Part_Number"
+F 6 " 603-RC0603FR-1010ML " H 5900 4400 50  0001 C CNN "Mouser Part Number"
 	1    5900 4400
 	-1   0    0    1
@@
 F 2 "Resistor_SMD:R_0603_1608Metric" H 6400 4400 50  0001 C CNN
 F 3 "~" H 6400 4400 50  0001 C CNN
-F 4 "Vishay" H 6400 4400 50  0001 C CNN "Manufacturer_Name"
-F 5 "CRCW060310M0FKEAC" H 6400 4400 50  0001 C CNN "Manufacturer_Part_Number"
-F 6 " 71-CRCW060310M0FKEAC " H 6400 4400 50  0001 C CNN "Mouser Part Number"
+F 4 "Yageo" H 6400 4400 50  0001 C CNN "Manufacturer_Name"
+F 5 "RC0603FR-1010ML" H 6400 4400 50  0001 C CNN "Manufacturer_Part_Number"
+F 6 " 603-RC0603FR-1010ML " H 6400 4400 50  0001 C CNN "Mouser Part Number"
 	1    6400 4400
 	-1   0    0    1
@@
 F 2 "Capacitor_SMD:C_0603_1608Metric" H 6700 4400 50  0001 C CNN
 F 3 "~" H 6700 4400 50  0001 C CNN
+F 4 "AVX" H 6700 4400 50  0001 C CNN "Manufacturer_Name"
+F 5 "0603YC104MAT4A" H 6700 4400 50  0001 C CNN "Manufacturer_Part_Number"
+F 6 "581-0603YC104MAT4A" H 6700 4400 50  0001 C CNN "Mouser Part Number"
 	1    6700 4400
 	1    0    0    -1
