File: pcb/senior_project_pcb/power.sch (KiCad schematic (older format))
At the start: 26 parts, among them Q1 Q_DUAL_NMOS, U1 stm32wb55ccu6, U3 MCP73831-2-OT, U4 AP9101CK6, U5 MIC5504-3.3YM5

Commit message: Add pulse oximeter circuit
Parts:
- added C14, C15: 1u, Capacitor_SMD:C_0603_1608Metric, symbol Device:C_Small
- added J2: USB_B_Micro, symbol Connector:USB_B_Micro
- added U2: MIC5504-1.8YM5, Package_TO_SOT_SMD:SOT-23-5, symbol Regulator_Linear:MIC5504-1.8YM5
Connections:
- net labels added: +1V8, USB_D+, USB_D-
- wire segments 48 -> 58
- no-connect marks 0 -> 1
Other:
- note added: "1.8V rail regulation\n"
- moved on the sheet: C12, C13, U5

Commit message: Connect up the pulse oximeter and USB
Parts:
- J2: footprint (none) -> Connector_USB:USB_Micro-AB_Molex_47590-0001
Changed lines of the file:
@@
 F 0 "J2" H 5307 2217 50  0000 C CNN
 F 1 "USB_B_Micro" H 5307 2126 50  0000 C CNN
-F 2 "" H 5400 1700 50  0001 C CNN
+F 2 "Connector_USB:USB_Micro-AB_Molex_47590-0001" H 5400 1700 50  0001 C CNN
 F 3 "~" H 5400 1700 50  0001 C CNN
 	1    5250 1750

Commit message: Add temp sensor
Parts:
- BT1: footprint Capacitor_SMD:C_0603_1608Metric -> Connector_JST:JST_EH_S2B-EH_1x02_P2.50mm_Horizontal
Connections:
- net labels added: +3.3VA
- wire segments 58 -> 59
Other:
- note added: "Analog supply filtering"
- moved on the sheet: C3, L1
Changed lines of the file:
@@
 $Descr A4 11693 8268
 encoding utf-8
-Sheet 2 5
+Sheet 2 6
 Title ""
 Date ""
@@
 L power:+3.3V #PWR01
 U 1 1 5FB08B14
-P 7550 5050
-F 0 "#PWR01" H 7550 4900 50  0001 C CNN
-F 1 "+3.3V" H 7565 5223 50  0000 C CNN
-F 2 "" H 7550 5050 50  0001 C CNN
-F 3 "" H 7550 5050 50  0001 C CNN
-	1    7550 5050
+P 4500 4300
+F 0 "#PWR01" H 4500 4150 50  0001 C CNN
+F 1 "+3.3V" H 4515 4473 50  0000 C CNN
+F 2 "" H 4500 4300 50  0001 C CNN
+F 3 "" H 4500 4300 50  0001 C CNN
+	1    4500 4300
 	1    0    0    -1
 $EndComp
@@
 L Device:L_Small L1
 U 1 1 5FB095DF
-P 7800 5050
-F 0 "L1" V 7619 5050 50  0000 C CNN
-F 1 "L_Small" V 7710 5050 50  0000 C CNN
-F 2 "Inductor_SMD:L_0805_2012Metric" H 7800 5050 50  0001 C CNN
-F 3 "~" H 7800 5050 50  0001 C CNN
-	1    7800 5050
+P 4750 4300
+F 0 "L1" V 4569 4300 50  0000 C CNN
+F 1 "L_Small" V 4660 4300 50  0000 C CNN
+F 2 "Inductor_SMD:L_0805_2012Metric" H 4750 4300 50  0001 C CNN
+F 3 "~" H 4750 4300 50  0001 C CNN
+	1    4750 4300
 	0    1    1    0
 $EndComp
@@
 L Device:C_Small C3
 U 1 1 5FB09C36
-P 8000 5150
-F 0 "C3" H 8092 5196 50  0000 L CNN
-F 1 "100n" H 8092 5105 50  0000 L CNN
-F 2 "Capacitor_SMD:C_0603_1608Metric" H 8000 5150 50  0001 C CNN
-F 3 "~" H 8000 5150 50  0001 C CNN
-	1    8000 5150
+P 4950 4400
+F 0 "C3" H 5042 4446 50  0000 L CNN
+F 1 "100n" H 5042 4355 50  0000 L CNN
+F 2 "Capacitor_SMD:C_0603_1608Metric" H 4950 4400 50  0001 C CNN
+F 3 "~" H 4950 4400 50  0001 C CNN
+	1    4950 4400
 	1    0    0    -1
 $EndComp
@@
 L power:GND #PWR04
 U 1 1 5FB0A681
-P 8000 5250
-F 0 "#PWR04" H 8000 5000 50  0001 C CNN
-F 1 "GND" H 8005 5077 50  0000 C CNN
-F 2 "" H 8000 5250 50  0001 C CNN
-F 3 "" H 8000 5250 50  0001 C CNN
-	1    8000 5250
-	1    0    0    -1
-$EndComp
-Wire Wire Line
-	7550 5050 7700 5050
-Wire Wire Line
-	7900 5050 8000 5050
-Connection ~ 8000 5050
-Wire Wire Line
-	8000 5050 8300 5050
+P 4950 4500
+F 0 "#PWR04" H 4950 4250 50  0001 C CNN
+F 1 "GND" H 4955 4327 50  0000 C CNN
+F 2 "" H 4950 4500 50  0001 C CNN
+F 3 "" H 4950 4500 50  0001 C CNN
+	1    4950 4500
+	1    0    0    -1
+$EndComp
+Wire Wire Line
+	4500 4300 4650 4300
+Wire Wire Line
+	4850 4300 4950 4300
+Connection ~ 4950 4300
+Wire Wire Line
+	4950 4300 5200 4300
 $Comp
 L power:+3.3V #PWR02
@@
 F 0 "BT1" H 750 2250 50  0000 L CNN
 F 1 "Battery_Cell" H 700 2150 50  0000 L CNN
-F 2 "Capacitor_SMD:C_0603_1608Metric" V 1000 2260 50  0001 C CNN
+F 2 "Connector_JST:JST_EH_S2B-EH_1x02_P2.50mm_Horizontal" V 1000 2260 50  0001 C CNN
 F 3 "~" V 1000 2260 50  0001 C CNN
 	1    1000 2200
@@
 3.3V rail regulation\n
 $Comp
-L Device:Q_DUAL_NMOS_S1G1D2S2G2D1 Q1
-U 2 1 5FC51F70
-P 2150 2850
-F 0 "Q1" H 2355 2896 50  0000 L CNN
-F 1 "Q_DUAL_NMOS" H 2355 2805 50  0000 L CNN
-F 2 "Package_TO_SOT_SMD:SOT-363_SC-70-6" H 2350 2850 50  0001 C CNN
-F 3 "~" H 2350 2850 50  0001 C CNN
-	2    2150 2850
-	-1   0    0    -1
-$EndComp
-$Comp
-L Device:Q_DUAL_NMOS_S1G1D2S2G2D1 Q1
-U 1 1 5FC5EF4A
-P 2150 2250
-F 0 "Q1" H 2355 2204 50  0000 L CNN
-F 1 "Q_DUAL_NMOS" H 2355 2295 50  0000 L CNN
-F 2 "Package_TO_SOT_SMD:SOT-363_SC-70-6" H 2350 2250 50  0001 C CNN
-F 3 "~" H 2350 2250 50  0001 C CNN
-	1    2150 2250
-	-1   0    0    1
-$EndComp
-$Comp
 L Regulator_Linear:MIC5504-1.8YM5 U2
 U 1 1 6017A0E8
@@
 $EndComp
 $Comp
-L power:+BATT #PWR028
-U 1 1 601A01C2
-P 3550 6000
-F 0 "#PWR028" H 3550 5850 50  0001 C CNN
-F 1 "+BATT" H 3565 6173 50  0000 C CNN
-F 2 "" H 3550 6000 50  0001 C CNN
-F 3 "" H 3550 6000 50  0001 C CNN
-	1    3550 6000
-	1    0    0    -1
-$EndComp
-$Comp
 L power:GND #PWR029
 U 1 1 601A0BBF
@@
 Wire Wire Line
 	3550 6000 3900 6000
-Connection ~ 3550 6000
 Wire Wire Line
 	4000 6200 3900 6200
@@
 	1    0    0    -1
 $EndComp
-Text HLabel 5750 1750 2    50   Input ~ 0
+Text HLabel 5750 1750 2    50   BiDi ~ 0
 USB_D+
-Text HLabel 5750 1850 2    50   Input ~ 0
+Text HLabel 5750 1850 2    50   BiDi ~ 0
 USB_D-
 Wire Wire Line
@@
 	2050 1900 2300 1900
 $Comp
-L power:PWR_FLAG #FLG0102
-U 1 1 6024A7EF
-P 8300 5050
-F 0 "#FLG0102" H 8300 5125 50  0001 C CNN
-F 1 "PWR_FLAG" H 8300 5223 50  0000 C CNN
-F 2 "" H 8300 5050 50  0001 C CNN
-F 3 "~" H 8300 5050 50  0001 C CNN
-	1    8300 5050
-	1    0    0    -1
-$EndComp
-Connection ~ 8300 5050
-Wire Wire Line
-	8300 5050 8550 5050
-$Comp
 L power:PWR_FLAG #FLG0103
 U 1 1 60280195
@@
 Wire Wire Line
 	1000 2350 1000 2300
+$Comp
+L power:+3.3VA #PWR0116
+U 1 1 601608E8
+P 5650 4300
+F 0 "#PWR0116" H 5650 4150 50  0001 C CNN
+F 1 "+3.3VA" H 5665 4473 50  0000 C CNN
+F 2 "" H 5650 4300 50  0001 C CNN
+F 3 "" H 5650 4300 50  0001 C CNN
+	1    5650 4300
+	1    0    0    -1
+$EndComp
+$Comp
+L power:PWR_FLAG #FLG0102
+U 1 1 6016133A
+P 5200 4300
+F 0 "#FLG0102" H 5200 4375 50  0001 C CNN
+F 1 "PWR_FLAG" H 5200 4473 50  0000 C CNN
+F 2 "" H 5200 4300 50  0001 C CNN
+F 3 "~" H 5200 4300 50  0001 C CNN
+	1    5200 4300
+	1    0    0    -1
+$EndComp
+Connection ~ 5200 4300
+Wire Wire Line
+	5200 4300 5650 4300
+$Comp
+L power:+3.3VA #PWR0117
+U 1 1 6016B0B3
+P 8350 5050
+F 0 "#PWR0117" H 8350 4900 50  0001 C CNN
+F 1 "+3.3VA" H 8365 5223 50  0000 C CNN
+F 2 "" H 8350 5050 50  0001 C CNN
+F 3 "" H 8350 5050 50  0001 C CNN
+	1    8350 5050
+	1    0    0    -1
+$EndComp
+Wire Wire Line
+	8350 5050 8550 5050
+Wire Notes Line
+	4300 3850 5900 3850
+Wire Notes Line
+	5900 3850 5900 5350
+Wire Notes Line
+	5900 5350 4300 5350
+Wire Notes Line
+	4300 5350 4300 3850
+Text Notes 4300 3750 0    50   ~ 0
+Analog supply filtering
+$Comp
+L Device:Q_DUAL_NMOS_S1G1D2S2G2D1 Q1
+U 1 1 5FC51F70
+P 2150 2850
+F 0 "Q1" H 2355 2896 50  0000 L CNN
+F 1 "Q_DUAL_NMOS" H 2355 2805 50  0000 L CNN
+F 2 "Package_TO_SOT_SMD:SOT-363_SC-70-6" H 2350 2850 50  0001 C CNN
+F 3 "~" H 2350 2850 50  0001 C CNN
+	1    2150 2850
+	-1   0    0    -1
+$EndComp
+$Comp
+L Device:Q_DUAL_NMOS_S1G1D2S2G2D1 Q1
+U 2 1 5FC5EF4A
+P 2150 2250
+F 0 "Q1" H 2355 2204 50  0000 L CNN
+F 1 "Q_DUAL_NMOS" H 2355 2295 50  0000 L CNN
+F 2 "Package_TO_SOT_SMD:SOT-363_SC-70-6" H 2350 2250 50  0001 C CNN
+F 3 "~" H 2350 2250 50  0001 C CNN
+	2    2150 2250
+	-1   0    0    1
+$EndComp
+$Comp
+L power:+3.3V #PWR?
+U 1 1 60199BB8
+P 3550 6000
+F 0 "#PWR?" H 3550 5850 50  0001 C CNN
+F 1 "+3.3V" H 3565 6173 50  0000 C CNN
+F 2 "" H 3550 6000 50  0001 C CNN
+F 3 "" H 3550 6000 50  0001 C CNN
+	1    3550 6000
+	1    0    0    -1
+$EndComp
+Connection ~ 3550 6000
 $EndSCHEMATC

Commit message: Initial layout mostly done
Parts:
- removed C15: 1u, Capacitor_SMD:C_0603_1608Metric, symbol Device:C_Small
- removed C6, C7: 100n, Capacitor_SMD:C_0603_1608Metric, symbol Device:C_Small
- removed U2: MIC5504-1.8YM5, Package_TO_SOT_SMD:SOT-23-5, symbol Regulator_Linear:MIC5504-1.8YM5
- C14: value 1u -> 100n
Connections:
- net labels removed: +1V8
- wire segments 59 -> 51
Other:
- note removed: "1.8V rail regulation\n"
Changed lines of the file:
@@
-$EndComp
-$Comp
-L Device:C_Small C6
-U 1 1 5FB0DB92
-P 8600 3800
-F 0 "C6" H 8550 3500 50  0000 L CNN
-F 1 "100n" H 8500 3600 50  0000 L CNN
-F 2 "Capacitor_SMD:C_0603_1608Metric" H 8600 3800 50  0001 C CNN
-F 3 "~" H 8600 3800 50  0001 C CNN
-	1    8600 3800
-	1    0    0    -1
-$EndComp
-$Comp
-L Device:C_Small C7
-U 1 1 5FB0E09D
-P 8800 3800
-F 0 "C7" H 8750 3500 50  0000 L CNN
-F 1 "100n" H 8700 3600 50  0000 L CNN
-F 2 "Capacitor_SMD:C_0603_1608Metric" H 8800 3800 50  0001 C CNN
-F 3 "~" H 8800 3800 50  0001 C CNN
-	1    8800 3800
-	1    0    0    -1
 $EndComp
 $Comp
@@
 	8200 3700 8400 3700
 Connection ~ 8400 3700
-Wire Wire Line
-	8400 3700 8600 3700
-Connection ~ 8600 3700
-Wire Wire Line
-	8600 3700 8800 3700
-Connection ~ 8800 3700
-Wire Wire Line
-	8800 3700 9000 3700
-Wire Wire Line
-	9000 3900 8800 3900
 Connection ~ 7800 3900
 Connection ~ 8000 3900
@@
 Wire Wire Line
 	8400 3900 8200 3900
-Connection ~ 8600 3900
-Wire Wire Line
-	8600 3900 8400 3900
-Connection ~ 8800 3900
-Wire Wire Line
-	8800 3900 8600 3900
 $Comp
 L Device:C_Small C9
@@
 Text Notes 600  5500 0    50   ~ 0
 3.3V rail regulation\n
-$Comp
-L Regulator_Linear:MIC5504-1.8YM5 U2
-U 1 1 6017A0E8
-P 4400 6100
-F 0 "U2" H 4400 6467 50  0000 C CNN
-F 1 "MIC5504-1.8YM5" H 4400 6376 50  0000 C CNN
-F 2 "Package_TO_SOT_SMD:SOT-23-5" H 4400 5700 50  0001 C CNN
-F 3 "http://ww1.microchip.com/downloads/en/DeviceDoc/MIC550X.pdf" H 4150 6350 50  0001 C CNN
-	1    4400 6100
-	1    0    0    -1
-$EndComp
 Wire Notes Line
 	2900 5650 2900 6750
@@
 Wire Notes Line
 	650  5650 2900 5650
-$Comp
-L Device:C_Small C14
-U 1 1 6019ED6A
-P 3550 6100
-F 0 "C14" H 3642 6146 50  0000 L CNN
-F 1 "1u" H 3642 6055 50  0000 L CNN
-F 2 "Capacitor_SMD:C_0603_1608Metric" H 3550 6100 50  0001 C CNN
-F 3 "~" H 3550 6100 50  0001 C CNN
-	1    3550 6100
-	1    0    0    -1
-$EndComp
-$Comp
-L Device:C_Small C15
-U 1 1 6019F7FB
-P 5150 6100
-F 0 "C15" H 5242 6146 50  0000 L CNN
-F 1 "1u" H 5242 6055 50  0000 L CNN
-F 2 "Capacitor_SMD:C_0603_1608Metric" H 5150 6100 50  0001 C CNN
-F 3 "~" H 5150 6100 50  0001 C CNN
-	1    5150 6100
-	1    0    0    -1
-$EndComp
-$Comp
-L power:GND #PWR029
-U 1 1 601A0BBF
-P 3550 6200
-F 0 "#PWR029" H 3550 5950 50  0001 C CNN
-F 1 "GND" H 3555 6027 50  0000 C CNN
-F 2 "" H 3550 6200 50  0001 C CNN
-F 3 "" H 3550 6200 50  0001 C CNN
-	1    3550 6200
-	1    0    0    -1
-$EndComp
-Wire Wire Line
-	3550 6000 3900 6000
-Wire Wire Line
-	4000 6200 3900 6200
-Wire Wire Line
-	3900 6200 3900 6000
-Connection ~ 3900 6000
-Wire Wire Line
-	3900 6000 4000 6000
-$Comp
-L power:GND #PWR030
-U 1 1 601A654F
-P 4400 6400
-F 0 "#PWR030" H 4400 6150 50  0001 C CNN
-F 1 "GND" H 4405 6227 50  0000 C CNN
-F 2 "" H 4400 6400 50  0001 C CNN
-F 3 "" H 4400 6400 50  0001 C CNN
-	1    4400 6400
-	1    0    0    -1
-$EndComp
-$Comp
-L power:GND #PWR032
-U 1 1 601A6E8A
-P 5150 6200
-F 0 "#PWR032" H 5150 5950 50  0001 C CNN
-F 1 "GND" H 5155 6027 50  0000 C CNN
-F 2 "" H 5150 6200 50  0001 C CNN
-F 3 "" H 5150 6200 50  0001 C CNN
-	1    5150 6200
-	1    0    0    -1
-$EndComp
-$Comp
-L power:+1V8 #PWR031
-U 1 1 601B8895
-P 5150 6000
-F 0 "#PWR031" H 5150 5850 50  0001 C CNN
-F 1 "+1V8" H 5165 6173 50  0000 C CNN
-F 2 "" H 5150 6000 50  0001 C CNN
-F 3 "" H 5150 6000 50  0001 C CNN
-	1    5150 6000
-	1    0    0    -1
-$EndComp
-Connection ~ 5150 6000
-Text Notes 3400 5550 0    50   ~ 0
-1.8V rail regulation\n
-Wire Notes Line
-	5550 5650 5550 6750
-Wire Notes Line
-	5550 6750 3300 6750
-Wire Notes Line
-	3300 6750 3300 5650
-Wire Notes Line
-	3300 5650 5550 5650
 $Comp
 L power:+BATT #PWR0104
@@
 Wire Wire Line
 	2000 6000 2550 6000
-Wire Wire Line
-	4800 6000 5150 6000
 Wire Wire Line
 	5550 1550 5800 1550
@@
 Connection ~ 5200 4300
 Wire Wire Line
-	5200 4300 5650 4300
+	5200 4300 5400 4300
 $Comp
 L power:+3.3VA #PWR0117
@@
 $EndComp
 $Comp
-L power:+3.3V #PWR?
-U 1 1 60199BB8
-P 3550 6000
-F 0 "#PWR?" H 3550 5850 50  0001 C CNN
-F 1 "+3.3V" H 3565 6173 50  0000 C CNN
-F 2 "" H 3550 6000 50  0001 C CNN
-F 3 "" H 3550 6000 50  0001 C CNN
-	1    3550 6000
-	1    0    0    -1
-$EndComp
-Connection ~ 3550 6000
+L Device:C_Small C14
+U 1 1 60318B80
+P 5400 4400
+F 0 "C14" H 5492 4446 50  0000 L CNN
+F 1 "100n" H 5492 4355 50  0000 L CNN
+F 2 "Capacitor_SMD:C_0603_1608Metric" H 5400 4400 50  0001 C CNN
+F 3 "~" H 5400 4400 50  0001 C CNN
+	1    5400 4400
+	1    0    0    -1
+$EndComp
+Connection ~ 5400 4300
+Wire Wire Line
+	5400 4300 5650 4300
+$Comp
+L power:GND #PWR030
+U 1 1 60319179
+P 5400 4500
+F 0 "#PWR030" H 5400 4250 50  0001 C CNN
+F 1 "GND" H 5405 4327 50  0000 C CNN
+F 2 "" H 5400 4500 50  0001 C CNN
+F 3 "" H 5400 4500 50  0001 C CNN
+	1    5400 4500
+	1    0    0    -1
+$EndComp
+Wire Wire Line
+	8400 3700 9000 3700
+Wire Wire Line
+	8400 3900 9000 3900
 $EndSCHEMATC

Commit message: Add ecg sensor
Parts:
- J2: symbol Connector:USB_B_Micro -> senior_project_pcb-rescue:USB_B_Micro-Connector
- U1: symbol stm32wb55cc:stm32wb55ccu6 -> senior_project_pcb-rescue:stm32wb55ccu6-stm32wb55cc
- U3: symbol Battery_Management:MCP73831-2-OT -> senior_project_pcb-rescue:MCP73831-2-OT-Battery_Management
- U4: symbol Battery_Management:AP9101CK6 -> senior_project_pcb-rescue:AP9101CK6-Battery_Management
Changed lines of the file:
@@
 EESchema Schematic File Version 4
-EELAYER 30 0
+LIBS:senior_project_pcb-cache
+EELAYER 29 0
 EELAYER END
 $Descr A4 11693 8268
 encoding utf-8
-Sheet 2 6
+Sheet 2 7
 Title ""
 Date ""
@@
 $EndComp
 $Comp
-L stm32wb55cc:stm32wb55ccu6 U1
+L senior_project_pcb-rescue:stm32wb55ccu6-stm32wb55cc U1
 U 2 1 5FB3EDF5
 P 9050 5400
@@
 $EndComp
 $Comp
-L Battery_Management:AP9101CK6 U4
+L senior_project_pcb-rescue:AP9101CK6-Battery_Management U4
 U 1 1 5FB508BD
 P 3150 2050
+AR Path="/5FB508BD" Ref="U4"  Part="1"
+AR Path="/5FB304C8/5FB508BD" Ref="U4"  Part="1"
 F 0 "U4" H 2600 2350 50  0000 C CNN
 F 1 "AP9101CK6" H 2500 2250 50  0000 C CNN
@@
 Microcontroller power connection\n
 $Comp
-L Battery_Management:MCP73831-2-OT U3
+L senior_project_pcb-rescue:MCP73831-2-OT-Battery_Management U3
 U 1 1 5FBBEA33
 P 2300 4550
@@
 $EndComp
 $Comp
-L Connector:USB_B_Micro J2
+L senior_project_pcb-rescue:USB_B_Micro-Connector J2
 U 1 1 60209B69
 P 5250 1750

Commit message: Add RF/Bluetooth to PCB
Parts:
- U1: symbol senior_project_pcb-rescue:stm32wb55ccu6-stm32wb55cc -> senior_project_pcb-rescue:stm32wb55ccu6-stm32wb55cc-senior_project_pcb-rescue
Changed lines of the file:
@@
 EESchema Schematic File Version 4
-LIBS:senior_project_pcb-cache
-EELAYER 29 0
+EELAYER 30 0
 EELAYER END
 $Descr A4 11693 8268
@@
 $EndComp
 $Comp
-L senior_project_pcb-rescue:stm32wb55ccu6-stm32wb55cc U1
+L senior_project_pcb-rescue:stm32wb55ccu6-stm32wb55cc-senior_project_pcb-rescue U1
 U 2 1 5FB3EDF5
 P 9050 5400

Commit message: PCB Update
Parts:
- removed J2: USB_B_Micro, Connector_USB:USB_Micro-AB_Molex_47590-0001, symbol senior_project_pcb-rescue:USB_B_Micro-Connector
- added J2: UJ2-MIBH2-4-SMT-TR, kicad_pretty:UJ2MIBH24SMTTR, symbol UJ2-MIBH2-4-SMT-TR:UJ2-MIBH2-4-SMT-TR
- added L3: 10n, Inductor_SMD:L_0402_1005Metric, symbol Device:L_Small
- added R29, R30: 22, Resistor_SMD:R_0603_1608Metric, symbol Device:R_Small
- BT1: footprint Connector_JST:JST_EH_S2B-EH_1x02_P2.50mm_Horizontal -> Connector_PinHeader_2.54mm:PinHeader_1x02_P2.54mm_Vertical
- C10, C9: Manufacturer_Name (none) -> Samsung; Manufacturer_Part_Number (none) -> CL10A475KP8NNNC; Mouser Part Number (none) -> 187-CL10A475KP8NNNC
- C12, C13: Manufacturer_Name (none) -> KEMET; Manufacturer_Part_Number (none) -> C0603C105K8PACTU; Mouser Part Number (none) -> 80-C0603C105K8P
- D1: footprint LED_SMD:LED_0603_1608Metric_Pad1.05x0.95mm_HandSolder -> LED_SMD:LED_0603_1608Metric; Manufacturer_Name (none) -> Wurth Elektronik; Manufacturer_Part_Number (none) -> 150060RS75000; Mouser Part Number (none) -> 710-150060RS75000
- L1, L2: Manufacturer_Name (none) -> Murata Electronics; Manufacturer_Part_Number (none) -> LQM21FN100M70L; Mouser Part Number (none) -> 81-LQM21FN100M70L
- Q1: Manufacturer_Name (none) -> Nexperia; Manufacturer_Part_Number (none) -> BSS138BKS\\,115; Mouser Part Number (none) -> 771-BSS138BKS115
- R1: Manufacturer_Name (none) -> Yageo; Manufacturer_Part_Number (none) -> RC0603FR-0710KL; Mouser Part Number (none) -> 603-RC0603FR-0710KL
- R2: Manufacturer_Name (none) -> Vishay; Manufacturer_Part_Number (none) -> CRCW0603470RFKEAC; Mouser Part Number (none) -> 71-CRCW0603470RFKEAC
- R3: Manufacturer_Name (none) -> Vishay; Manufacturer_Part_Number (none) -> RCA0603300RFKEA; Mouser Part Number (none) -> 71-RCA0603300RFKEA
- R4: Manufacturer_Name (none) -> Vishay; Manufacturer_Part_Number (none) -> CRCW06032K70JNEAC; Mouser Part Number (none) -> 71-CRCW06032K70JNEAC
- U1: Manufacturer_Name (none) -> STMicro; Manufacturer_Part_Number (none) -> STM32WB55CEU6; Mouser Part Number (none) -> 511-STM32WB55CEU6
- U3: Manufacturer_Name (none) -> Microchip; Manufacturer_Part_Number (none) -> MCP73831T-2DCI/OT; Mouser Part Number (none) -> 579-MCP73831T-2DCIOT
- U4: Manufacturer_Name (none) -> Diodes Inc.; Manufacturer_Part_Number (none) -> AP9101CAK6-BVTRG1; Mouser Part Number (none) -> 621-AP9101CAK6BVTRG1
- U5: Manufacturer_Name (none) -> Microchip; Manufacturer_Part_Number (none) -> MIC5504-3.3YM5-TR; Mouser Part Number (none) -> 998-MIC5504-3.3YM5TR
Connections:
- net GND: now also J2.5, J2.MH1, J2.MH2, J2.MH3, J2.MH4
- net USB_D+: now also R29.1
- net USB_D-: now also R30.2
- net VBUS: now also J2.1
- net at L2.2: now also L3.2; no longer U1.33 (VLXSMPS)
- new net: L3.1, U1.33 (VLXSMPS)
- new net: J2.3, R29.2
- new net: J2.2, R30.1
