File: pcb/senior_project_pcb/power.sch (KiCad schematic (older format))
At the start: 29 parts, among them J2 UJ2-MIBH2-4-SMT-TR, Q1 Q_DUAL_NMOS, U1 stm32wb55ccu6, U3 MCP73831-2-OT, U4 AP9101CK6, U5 MIC5504-3.3YM5

Commit message: Send PCB off for manufacture
Parts:
- C1, C11, C14, C2, C3, C4, C5, C8: Manufacturer_Name (none) -> AVX; Manufacturer_Part_Number (none) -> 0603YC104MAT4A; Mouser Part Number (none) -> 581-0603YC104MAT4A
- L1, L2: Manufacturer_Name Murata Electronics -> Taiyo; Manufacturer_Part_Number LQM21FN100M70L -> LBR2012T100K; Mouser Part Number 81-LQM21FN100M70L -> 963-LBR2012T100K
- L3: Manufacturer_Part_Number LQG15WZ10NJ02D -> LQG15WH10NJ02D; Mouser Part Number 81-LQG15WZ10NJ02D -> 81-LQG15WH10NJ02D
- R2: Manufacturer_Name Vishay -> Yageo; Manufacturer_Part_Number CRCW0603470RFKEAC -> RC0603FR-10470RL; Mouser Part Number 71-CRCW0603470RFKEAC -> 603-RC0603FR-10470RL
- R3: Manufacturer_Name Vishay -> Yageo; Manufacturer_Part_Number RCA0603300RFKEA -> RC0603FR-10300RL; Mouser Part Number 71-RCA0603300RFKEA -> 603-RC0603FR-10300RL
- R4: Manufacturer_Name Vishay -> Yageo; Manufacturer_Part_Number CRCW06032K70JNEAC -> RC0603FR-072K7L; Mouser Part Number 71-CRCW06032K70JNEAC -> 603-RC0603FR-072K7L
- U4: Manufacturer_Part_Number AP9101CAK6-BVTRG1 -> AP9101CAK6-AYTRG1; Mouser Part Number 621-AP9101CAK6BVTRG1 -> 621-AP9101CAK6AYTRG1
Changed lines of the file:
@@
 F 2 "Inductor_SMD:L_0805_2012Metric" H 4750 4300 50  0001 C CNN
 F 3 "~" H 4750 4300 50  0001 C CNN
-F 4 "Murata Electronics" H 4750 4300 50  0001 C CNN "Manufacturer_Name"
-F 5 "LQM21FN100M70L " H 4750 4300 50  0001 C CNN "Manufacturer_Part_Number"
-F 6 "81-LQM21FN100M70L" H 4750 4300 50  0001 C CNN "Mouser Part Number"
+F 4 "Taiyo" H 4750 4300 50  0001 C CNN "Manufacturer_Name"
+F 5 "LBR2012T100K " H 4750 4300 50  0001 C CNN "Manufacturer_Part_Number"
+F 6 "963-LBR2012T100K" H 4750 4300 50  0001 C CNN "Mouser Part Number"
 	1    4750 4300
 	0    1    1    0
@@
 F 2 "Capacitor_SMD:C_0603_1608Metric" H 4950 4400 50  0001 C CNN
 F 3 "~" H 4950 4400 50  0001 C CNN
+F 4 "AVX" H 4950 4400 50  0001 C CNN "Manufacturer_Name"
+F 5 "0603YC104MAT4A" H 4950 4400 50  0001 C CNN "Manufacturer_Part_Number"
+F 6 "581-0603YC104MAT4A" H 4950 4400 50  0001 C CNN "Mouser Part Number"
 	1    4950 4400
 	1    0    0    -1
@@
 F 2 "Capacitor_SMD:C_0603_1608Metric" H 7800 3800 50  0001 C CNN
 F 3 "~" H 7800 3800 50  0001 C CNN
+F 4 "AVX" H 7800 3800 50  0001 C CNN "Manufacturer_Name"
+F 5 "0603YC104MAT4A" H 7800 3800 50  0001 C CNN "Manufacturer_Part_Number"
+F 6 "581-0603YC104MAT4A" H 7800 3800 50  0001 C CNN "Mouser Part Number"
 	1    7800 3800
 	1    0    0    -1
@@
 F 2 "Capacitor_SMD:C_0603_1608Metric" H 8000 3800 50  0001 C CNN
 F 3 "~" H 8000 3800 50  0001 C CNN
+F 4 "AVX" H 8000 3800 50  0001 C CNN "Manufacturer_Name"
+F 5 "0603YC104MAT4A" H 8000 3800 50  0001 C CNN "Manufacturer_Part_Number"
+F 6 "581-0603YC104MAT4A" H 8000 3800 50  0001 C CNN "Mouser Part Number"
 	1    8000 3800
 	1    0    0    -1
@@
 F 2 "Capacitor_SMD:C_0603_1608Metric" H 8200 3800 50  0001 C CNN
 F 3 "~" H 8200 3800 50  0001 C CNN
+F 4 "AVX" H 8200 3800 50  0001 C CNN "Manufacturer_Name"
+F 5 "0603YC104MAT4A" H 8200 3800 50  0001 C CNN "Manufacturer_Part_Number"
+F 6 "581-0603YC104MAT4A" H 8200 3800 50  0001 C CNN "Mouser Part Number"
 	1    8200 3800
 	1    0    0    -1
@@
 F 2 "Capacitor_SMD:C_0603_1608Metric" H 8400 3800 50  0001 C CNN
 F 3 "~" H 8400 3800 50  0001 C CNN
+F 4 "AVX" H 8400 3800 50  0001 C CNN "Manufacturer_Name"
+F 5 "0603YC104MAT4A" H 8400 3800 50  0001 C CNN "Manufacturer_Part_Number"
+F 6 "581-0603YC104MAT4A" H 8400 3800 50  0001 C CNN "Mouser Part Number"
 	1    8400 3800
 	1    0    0    -1
@@
 F 2 "Capacitor_SMD:C_0603_1608Metric" H 9000 3800 50  0001 C CNN
 F 3 "~" H 9000 3800 50  0001 C CNN
+F 4 "AVX" H 9000 3800 50  0001 C CNN "Manufacturer_Name"
+F 5 "0603YC104MAT4A" H 9000 3800 50  0001 C CNN "Manufacturer_Part_Number"
+F 6 "581-0603YC104MAT4A" H 9000 3800 50  0001 C CNN "Mouser Part Number"
 	1    9000 3800
 	1    0    0    -1
@@
 F 2 "Inductor_SMD:L_0805_2012Metric" H 9900 5200 50  0001 C CNN
 F 3 "~" H 9900 5200 50  0001 C CNN
-F 4 "Murata Electronics" H 9900 5200 50  0001 C CNN "Manufacturer_Name"
-F 5 "LQM21FN100M70L " H 9900 5200 50  0001 C CNN "Manufacturer_Part_Number"
-F 6 "81-LQM21FN100M70L" H 9900 5200 50  0001 C CNN "Mouser Part Number"
+F 4 "Taiyo" H 9900 5200 50  0001 C CNN "Manufacturer_Name"
+F 5 "LBR2012T100K" H 9900 5200 50  0001 C CNN "Manufacturer_Part_Number"
+F 6 "963-LBR2012T100K" H 9900 5200 50  0001 C CNN "Mouser Part Number"
 	1    9900 5200
 	-1   0    0    1
@@
 F 3 "https://www.diodes.com/assets/Datasheets/AP9101C.pdf" H 3150 2100 50  0001 C CNN
 F 4 "Diodes Inc." H 3150 2050 50  0001 C CNN "Manufacturer_Name"
-F 5 "AP9101CAK6-BVTRG1" H 3150 2050 50  0001 C CNN "Manufacturer_Part_Number"
-F 6 " 621-AP9101CAK6BVTRG1 " H 3150 2050 50  0001 C CNN "Mouser Part Number"
+F 5 "AP9101CAK6-AYTRG1" H 3150 2050 50  0001 C CNN "Manufacturer_Part_Number"
+F 6 " 621-AP9101CAK6AYTRG1 " H 3150 2050 50  0001 C CNN "Mouser Part Number"
 	1    3150 2050
 	-1   0    0    -1
@@
 F 2 "Capacitor_SMD:C_0603_1608Metric" H 3538 1150 50  0001 C CNN
 F 3 "~" H 3500 1300 50  0001 C CNN
+F 4 "AVX" H 3500 1300 50  0001 C CNN "Manufacturer_Name"
+F 5 "0603YC104MAT4A" H 3500 1300 50  0001 C CNN "Manufacturer_Part_Number"
+F 6 "581-0603YC104MAT4A" H 3500 1300 50  0001 C CNN "Mouser Part Number"
 	1    3500 1300
 	1    0    0    1
@@
 F 2 "Resistor_SMD:R_0603_1608Metric" V 3580 1150 50  0001 C CNN
 F 3 "~" H 3650 1150 50  0001 C CNN
-F 4 "Vishay" H 3650 1150 50  0001 C CNN "Manufacturer_Name"
-F 5 "RCA0603300RFKEA" H 3650 1150 50  0001 C CNN "Manufacturer_Part_Number"
-F 6 " 71-RCA0603300RFKEA " H 3650 1150 50  0001 C CNN "Mouser Part Number"
+F 4 "Yageo" H 3650 1150 50  0001 C CNN "Manufacturer_Name"
+F 5 "RC0603FR-10300RL" H 3650 1150 50  0001 C CNN "Manufacturer_Part_Number"
+F 6 "603-RC0603FR-10300RL" H 3650 1150 50  0001 C CNN "Mouser Part Number"
 	1    3650 1150
 	0    1    1    0
@@
 F 2 "Resistor_SMD:R_0603_1608Metric" V 3630 2200 50  0001 C CNN
 F 3 "~" H 3700 2200 50  0001 C CNN
-F 4 "Vishay" H 3700 2200 50  0001 C CNN "Manufacturer_Name"
-F 5 "CRCW06032K70JNEAC" H 3700 2200 50  0001 C CNN "Manufacturer_Part_Number"
-F 6 " 71-CRCW06032K70JNEAC " H 3700 2200 50  0001 C CNN "Mouser Part Number"
+F 4 "Yageo" H 3700 2200 50  0001 C CNN "Manufacturer_Name"
+F 5 "RC0603FR-072K7L" H 3700 2200 50  0001 C CNN "Manufacturer_Part_Number"
+F 6 "603-RC0603FR-072K7L" H 3700 2200 50  0001 C CNN "Mouser Part Number"
 	1    3700 2200
 	1    0    0    -1
@@
 F 2 "Resistor_SMD:R_0603_1608Metric" H 3300 4800 50  0001 C CNN
 F 3 "~" H 3300 4800 50  0001 C CNN
-F 4 "Vishay" H 3300 4800 50  0001 C CNN "Manufacturer_Name"
-F 5 "CRCW0603470RFKEAC" H 3300 4800 50  0001 C CNN "Manufacturer_Part_Number"
-F 6 " 71-CRCW0603470RFKEAC " H 3300 4800 50  0001 C CNN "Mouser Part Number"
+F 4 "Yageo" H 3300 4800 50  0001 C CNN "Manufacturer_Name"
+F 5 "RC0603FR-10470RL" H 3300 4800 50  0001 C CNN "Manufacturer_Part_Number"
+F 6 "603-RC0603FR-10470RL" H 3300 4800 50  0001 C CNN "Mouser Part Number"
 	1    3300 4800
 	1    0    0    -1
@@
 F 2 "Capacitor_SMD:C_0603_1608Metric" H 5400 4400 50  0001 C CNN
 F 3 "~" H 5400 4400 50  0001 C CNN
+F 4 "AVX" H 5400 4400 50  0001 C CNN "Manufacturer_Name"
+F 5 "0603YC104MAT4A" H 5400 4400 50  0001 C CNN "Manufacturer_Part_Number"
+F 6 "581-0603YC104MAT4A" H 5400 4400 50  0001 C CNN "Mouser Part Number"
 	1    5400 4400
 	1    0    0    -1
@@
 F 3 "~" H 9800 5100 50  0001 C CNN
 F 4 "Murata Electronics" H 9800 5100 50  0001 C CNN "Manufacturer_Name"
-F 5 "LQG15WZ10NJ02D " H 9800 5100 50  0001 C CNN "Manufacturer_Part_Number"
-F 6 " 81-LQG15WZ10NJ02D " H 9800 5100 50  0001 C CNN "Mouser Part Number"
+F 5 "LQG15WH10NJ02D" H 9800 5100 50  0001 C CNN "Manufacturer_Part_Number"
+F 6 "81-LQG15WH10NJ02D" H 9800 5100 50  0001 C CNN "Mouser Part Number"
 	1    9800 5100
 	0    -1   -1   0
