File: pcb/senior_project_pcb/pulse_oxy.sch (KiCad schematic (older format))
At the start: 9 parts, among them IC1 MAX30102, Q2 Q_DUAL_NMOS_S1G1D2S2G2D1

Commit message: Connect up the pulse oximeter and USB
Parts:
- C16, C17: footprint (none) -> Capacitor_SMD:C_0603_1608Metric
- Q2: footprint (none) -> Package_TO_SOT_SMD:SOT-363_SC-70-6
- R5, R6, R7, R8, R9: footprint (none) -> Resistor_SMD:R_0603_1608Metric
Changed lines of the file:
@@
 F 0 "Q2" V 5050 3300 50  0000 C CNN
 F 1 "Q_DUAL_NMOS_S1G1D2S2G2D1" V 5140 3300 50  0001 C CNN
-F 2 "" H 5000 3300 50  0001 C CNN
+F 2 "Package_TO_SOT_SMD:SOT-363_SC-70-6" H 5000 3300 50  0001 C CNN
 F 3 "~" H 5000 3300 50  0001 C CNN
 	1    4800 3300
@@
 F 0 "Q2" V 5500 3400 50  0000 C CNN
 F 1 "Q_DUAL_NMOS_S1G1D2S2G2D1" V 5590 3400 50  0001 C CNN
-F 2 "" H 5450 3400 50  0001 C CNN
+F 2 "Package_TO_SOT_SMD:SOT-363_SC-70-6" H 5450 3400 50  0001 C CNN
 F 3 "~" H 5450 3400 50  0001 C CNN
 	2    5250 3400
@@
 F 0 "R8" H 5659 3346 50  0000 L CNN
 F 1 "1k" H 5659 3255 50  0000 L CNN
-F 2 "" H 5600 3300 50  0001 C CNN
+F 2 "Resistor_SMD:R_0603_1608Metric" H 5600 3300 50  0001 C CNN
 F 3 "~" H 5600 3300 50  0001 C CNN
 	1    5600 3300
@@
 F 0 "R9" H 5859 3446 50  0000 L CNN
 F 1 "1k" H 5859 3355 50  0000 L CNN
-F 2 "" H 5800 3400 50  0001 C CNN
+F 2 "Resistor_SMD:R_0603_1608Metric" H 5800 3400 50  0001 C CNN
 F 3 "~" H 5800 3400 50  0001 C CNN
 	1    5800 3400
@@
 F 0 "R5" H 4159 3346 50  0000 L CNN
 F 1 "1k" H 4159 3255 50  0000 L CNN
-F 2 "" H 4100 3300 50  0001 C CNN
+F 2 "Resistor_SMD:R_0603_1608Metric" H 4100 3300 50  0001 C CNN
 F 3 "~" H 4100 3300 50  0001 C CNN
 	1    4100 3300
@@
 F 0 "R6" H 4409 3446 50  0000 L CNN
 F 1 "1k" H 4409 3355 50  0000 L CNN
-F 2 "" H 4350 3400 50  0001 C CNN
+F 2 "Resistor_SMD:R_0603_1608Metric" H 4350 3400 50  0001 C CNN
 F 3 "~" H 4350 3400 50  0001 C CNN
 	1    4350 3400
@@
 F 0 "R7" H 8459 3446 50  0000 L CNN
 F 1 "10k" H 8459 3355 50  0000 L CNN
-F 2 "" H 8400 3400 50  0001 C CNN
+F 2 "Resistor_SMD:R_0603_1608Metric" H 8400 3400 50  0001 C CNN
 F 3 "~" H 8400 3400 50  0001 C CNN
 	1    8400 3400
@@
 F 0 "C17" H 6192 4396 50  0000 L CNN
 F 1 "100n" H 6192 4305 50  0000 L CNN
-F 2 "" H 6100 4350 50  0001 C CNN
+F 2 "Capacitor_SMD:C_0603_1608Metric" H 6100 4350 50  0001 C CNN
 F 3 "~" H 6100 4350 50  0001 C CNN
 	1    6100 4350
@@
 F 0 "C16" H 5792 4396 50  0000 L CNN
 F 1 "100n" H 5792 4305 50  0000 L CNN
-F 2 "" H 5700 4350 50  0001 C CNN
+F 2 "Capacitor_SMD:C_0603_1608Metric" H 5700 4350 50  0001 C CNN
 F 3 "~" H 5700 4350 50  0001 C CNN
 	1    5700 4350

Commit message: Add temp sensor
Changed lines of the file:
@@
 $Descr A4 11693 8268
 encoding utf-8
-Sheet 5 5
+Sheet 5 6
 Title ""
 Date ""
@@
 	1    0    0    -1
 $EndComp
-Text HLabel 3800 3500 0    50   Input ~ 0
+Text HLabel 3800 3500 0    50   BiDi ~ 0
 SDA
-Text HLabel 3800 3400 0    50   Input ~ 0
+Text HLabel 3800 3400 0    50   BiDi ~ 0
 SCL
 $Comp
@@
 NoConn ~ 7950 3700
 NoConn ~ 7950 3800
-Text HLabel 8700 3500 2    50   Input ~ 0
+Text HLabel 8700 3500 2    50   Output ~ 0
 INT
 Wire Wire Line

Commit message: Initial layout mostly done
Parts:
- removed C16, C17: 100n, Capacitor_SMD:C_0603_1608Metric, symbol Device:C_Small
- removed IC1: MAX30102, OptoDevice:Maxim_OLGA-14_3.3x5.6mm_P0.8mm, symbol Sensor:MAX30102
- removed Q2: Q_DUAL_NMOS_S1G1D2S2G2D1, Package_TO_SOT_SMD:SOT-363_SC-70-6, symbol Device:Q_DUAL_NMOS_S1G1D2S2G2D1
- removed R8, R9: 1k, Resistor_SMD:R_0603_1608Metric, symbol Device:R_Small
- added J3: Conn_01x05, Connector_PinHeader_2.54mm:PinHeader_1x05_P2.54mm_Vertical, symbol Connector_Generic:Conn_01x05
- R5, R6: value 1k -> 2k
- R7: value 10k -> 2k
Connections:
- net labels added: +3V3
- net labels removed: +1V8
- wire segments 11 -> 7
- no-connect marks 2 -> 0
Other:
- note removed: "INT* can handle up to 5v and is open drain"

Commit message: Add ecg sensor
Parts:
- J3: symbol Connector_Generic:Conn_01x05 -> senior_project_pcb-rescue:Conn_01x05-Connector_Generic
Changed lines of the file:
@@
 EESchema Schematic File Version 4
-EELAYER 30 0
+LIBS:senior_project_pcb-cache
+EELAYER 29 0
 EELAYER END
 $Descr A4 11693 8268
 encoding utf-8
-Sheet 4 6
+Sheet 4 7
 Title ""
 Date ""
@@
 i2c 3.3v to 1.8v level shifter
 $Comp
-L Connector_Generic:Conn_01x05 J3
+L senior_project_pcb-rescue:Conn_01x05-Connector_Generic J3
 U 1 1 602CD835
 P 5400 3500

Commit message: Send PCB off for manufacture
Parts:
- R5, R6, R7: Manufacturer_Name (none) -> Yageo; Manufacturer_Part_Number (none) -> RC0603FR-072KL; Mouser Part Number (none) -> 603-RC0603FR-072KL
Changed lines of the file:
@@
 F 2 "Resistor_SMD:R_0603_1608Metric" H 4100 3300 50  0001 C CNN
 F 3 "~" H 4100 3300 50  0001 C CNN
+F 4 "Yageo" H 4100 3300 50  0001 C CNN "Manufacturer_Name"
+F 5 "RC0603FR-072KL" H 4100 3300 50  0001 C CNN "Manufacturer_Part_Number"
+F 6 "603-RC0603FR-072KL" H 4100 3300 50  0001 C CNN "Mouser Part Number"
 	1    4100 3300
 	1    0    0    -1
@@
 F 2 "Resistor_SMD:R_0603_1608Metric" H 4350 3400 50  0001 C CNN
 F 3 "~" H 4350 3400 50  0001 C CNN
+F 4 "Yageo" H 4350 3400 50  0001 C CNN "Manufacturer_Name"
+F 5 "RC0603FR-072KL" H 4350 3400 50  0001 C CNN "Manufacturer_Part_Number"
+F 6 "603-RC0603FR-072KL" H 4350 3400 50  0001 C CNN "Mouser Part Number"
 	1    4350 3400
 	1    0    0    -1
@@
 F 2 "Resistor_SMD:R_0603_1608Metric" H 4700 3200 50  0001 C CNN
 F 3 "~" H 4700 3200 50  0001 C CNN
+F 4 "Yageo" H 4700 3200 50  0001 C CNN "Manufacturer_Name"
+F 5 "RC0603FR-072KL" H 4700 3200 50  0001 C CNN "Manufacturer_Part_Number"
+F 6 "603-RC0603FR-072KL" H 4700 3200 50  0001 C CNN "Mouser Part Number"
 	1    4700 3200
 	1    0    0    -1
