File: pcb/senior_project_pcb/temp_sensor.sch (KiCad schematic (older format))
At the start: 9 parts, among them IC2 ZTP-148SRC1, U6 AD8539

Commit message: Add ecg sensor
Parts:
- IC2: symbol ZTP-148SRC1:ZTP-148SRC1 -> senior_project_pcb-rescue:ZTP-148SRC1-ZTP-148SRC1
Changed lines of the file:
@@
 EESchema Schematic File Version 4
-EELAYER 30 0
+LIBS:senior_project_pcb-cache
+EELAYER 29 0
 EELAYER END
 $Descr A4 11693 8268
 encoding utf-8
-Sheet 5 6
+Sheet 5 7
 Title ""
 Date ""
@@
 $EndDescr
 $Comp
-L ZTP-148SRC1:ZTP-148SRC1 IC2
+L senior_project_pcb-rescue:ZTP-148SRC1-ZTP-148SRC1 IC2
 U 1 1 601471B4
 P 4350 3750

Commit message: PCB Update
Parts:
- R12: value 100k -> 100k 1%; Manufacturer_Name (none) -> Vishay; Manufacturer_Part_Number (none) -> CRCW0603100KFKEAC; Mouser Part Number (none) -> 71-CRCW0603100KFKEAC
- R13, R14: value 10k -> 10k 1%; Manufacturer_Name (none) -> Yageo; Manufacturer_Part_Number (none) -> RC0603FR-0710KL; Mouser Part Number (none) -> 603-RC0603FR-0710KL
- R15: value 100 -> 12 1%; Manufacturer_Name (none) -> Bourns; Manufacturer_Part_Number (none) -> CR0603-FX-12R0ELF; Mouser Part Number (none) -> 652-CR0603FX-12R0ELF
- R16: value 49.9k -> 33k 1%; Manufacturer_Name (none) -> Bourns; Manufacturer_Part_Number (none) -> CR0603-FX-3302ELF; Mouser Part Number (none) -> 652-CR0603FX-3302ELF
- U6: Manufacturer_Name (none) -> Analog; Manufacturer_Part_Number (none) -> AD8539ARMZ; Mouser Part Number (none) -> 584-AD8539ARMZ
Changed lines of the file:
@@
 P 2950 3550
 F 0 "R12" H 3020 3596 50  0000 L CNN
-F 1 "100k" H 3020 3505 50  0000 L CNN
+F 1 "100k 1%" H 3020 3505 50  0000 L CNN
 F 2 "Resistor_SMD:R_0603_1608Metric" V 2880 3550 50  0001 C CNN
 F 3 "~" H 2950 3550 50  0001 C CNN
+F 4 "Vishay" H 2950 3550 50  0001 C CNN "Manufacturer_Name"
+F 5 "CRCW0603100KFKEAC" H 2950 3550 50  0001 C CNN "Manufacturer_Part_Number"
+F 6 " 71-CRCW0603100KFKEAC " H 2950 3550 50  0001 C CNN "Mouser Part Number"
 	1    2950 3550
 	1    0    0    -1
@@
 F 2 "Package_SO:MSOP-8_3x3mm_P0.65mm" H 3900 5550 50  0001 C CNN
 F 3 "~" H 3900 5550 50  0001 C CNN
+F 4 "Analog" H 3900 5550 50  0001 C CNN "Manufacturer_Name"
+F 5 "AD8539ARMZ" H 3900 5550 50  0001 C CNN "Manufacturer_Part_Number"
+F 6 "584-AD8539ARMZ" H 3900 5550 50  0001 C CNN "Mouser Part Number"
 	1    3900 5550
 	1    0    0    -1
@@
 F 2 "Package_SO:MSOP-8_3x3mm_P0.65mm" H 6450 3800 50  0001 C CNN
 F 3 "~" H 6450 3800 50  0001 C CNN
+F 4 "Analog" H 6450 3800 50  0001 C CNN "Manufacturer_Name"
+F 5 "AD8539ARMZ" H 6450 3800 50  0001 C CNN "Manufacturer_Part_Number"
+F 6 "584-AD8539ARMZ" H 6450 3800 50  0001 C CNN "Mouser Part Number"
 	2    6450 3800
 	1    0    0    -1
@@
 F 2 "Package_SO:MSOP-8_3x3mm_P0.65mm" H 2150 5550 50  0001 C CNN
 F 3 "~" H 2150 5550 50  0001 C CNN
+F 4 "Analog" H 2150 5550 50  0001 C CNN "Manufacturer_Name"
+F 5 "AD8539ARMZ" H 2150 5550 50  0001 C CNN "Manufacturer_Part_Number"
+F 6 "584-AD8539ARMZ" H 2150 5550 50  0001 C CNN "Mouser Part Number"
 	3    2150 5550
 	1    0    0    -1
@@
 P 2850 5300
 F 0 "R13" H 2920 5346 50  0000 L CNN
-F 1 "10k" H 2920 5255 50  0000 L CNN
+F 1 "10k 1%" H 2920 5255 50  0000 L CNN
 F 2 "Resistor_SMD:R_0603_1608Metric" V 2780 5300 50  0001 C CNN
 F 3 "~" H 2850 5300 50  0001 C CNN
+F 4 "Yageo" H 2850 5300 50  0001 C CNN "Manufacturer_Name"
+F 5 "RC0603FR-0710KL" H 2850 5300 50  0001 C CNN "Manufacturer_Part_Number"
+F 6 "603-RC0603FR-0710KL" H 2850 5300 50  0001 C CNN "Mouser Part Number"
 	1    2850 5300
 	1    0    0    -1
@@
 P 2850 5600
 F 0 "R14" H 2920 5646 50  0000 L CNN
-F 1 "10k" H 2920 5555 50  0000 L CNN
+F 1 "10k 1%" H 2920 5555 50  0000 L CNN
 F 2 "Resistor_SMD:R_0603_1608Metric" V 2780 5600 50  0001 C CNN
 F 3 "~" H 2850 5600 50  0001 C CNN
+F 4 "Yageo" H 2850 5600 50  0001 C CNN "Manufacturer_Name"
+F 5 "RC0603FR-0710KL" H 2850 5600 50  0001 C CNN "Manufacturer_Part_Number"
+F 6 "603-RC0603FR-0710KL" H 2850 5600 50  0001 C CNN "Mouser Part Number"
 	1    2850 5600
 	1    0    0    -1
@@
 P 6450 4200
 F 0 "R16" V 6243 4200 50  0000 C CNN
-F 1 "49.9k" V 6334 4200 50  0000 C CNN
+F 1 "33k 1%" V 6334 4200 50  0000 C CNN
 F 2 "Resistor_SMD:R_0603_1608Metric" V 6380 4200 50  0001 C CNN
 F 3 "~" H 6450 4200 50  0001 C CNN
+F 4 "Bourns" H 6450 4200 50  0001 C CNN "Manufacturer_Name"
+F 5 "CR0603-FX-3302ELF" H 6450 4200 50  0001 C CNN "Manufacturer_Part_Number"
+F 6 " 652-CR0603FX-3302ELF " H 6450 4200 50  0001 C CNN "Mouser Part Number"
 	1    6450 4200
 	0    1    1    0
@@
 P 6050 4350
 F 0 "R15" H 5980 4304 50  0000 R CNN
-F 1 "100" H 5980 4395 50  0000 R CNN
+F 1 "12 1%" H 5980 4395 50  0000 R CNN
 F 2 "Resistor_SMD:R_0603_1608Metric" V 5980 4350 50  0001 C CNN
 F 3 "~" H 6050 4350 50  0001 C CNN
+F 4 "Bourns" H 6050 4350 50  0001 C CNN "Manufacturer_Name"
+F 5 "CR0603-FX-12R0ELF" H 6050 4350 50  0001 C CNN "Manufacturer_Part_Number"
+F 6 " 652-CR0603FX-12R0ELF " H 6050 4350 50  0001 C CNN "Mouser Part Number"
 	1    6050 4350
 	-1   0    0    1

Commit message: Send PCB off for manufacture
Parts:
- C18, C19: Manufacturer_Name (none) -> AVX; Manufacturer_Part_Number (none) -> 0603YC104MAT4A; Mouser Part Number (none) -> 581-0603YC104MAT4A
- R12: Manufacturer_Name Vishay -> Yageo; Manufacturer_Part_Number CRCW0603100KFKEAC -> RC0603FR-13100KL; Mouser Part Number 71-CRCW0603100KFKEAC -> 603-RC0603FR-13100KL
- R15: Manufacturer_Name Bourns -> Yageo; Manufacturer_Part_Number CR0603-FX-12R0ELF -> RC0603FR-0712RL; Mouser Part Number 652-CR0603FX-12R0ELF -> 603-RC0603FR-0712RL
- R16: Manufacturer_Name Bourns -> Yageo; Manufacturer_Part_Number CR0603-FX-3302ELF -> RC0603FR-0733KL; Mouser Part Number 652-CR0603FX-3302ELF -> 603-RC0603FR-0733KL
Changed lines of the file:
@@
 F 2 "Resistor_SMD:R_0603_1608Metric" V 2880 3550 50  0001 C CNN
 F 3 "~" H 2950 3550 50  0001 C CNN
-F 4 "Vishay" H 2950 3550 50  0001 C CNN "Manufacturer_Name"
-F 5 "CRCW0603100KFKEAC" H 2950 3550 50  0001 C CNN "Manufacturer_Part_Number"
-F 6 " 71-CRCW0603100KFKEAC " H 2950 3550 50  0001 C CNN "Mouser Part Number"
+F 4 "Yageo" H 2950 3550 50  0001 C CNN "Manufacturer_Name"
+F 5 "RC0603FR-13100KL" H 2950 3550 50  0001 C CNN "Manufacturer_Part_Number"
+F 6 " 603-RC0603FR-13100KL " H 2950 3550 50  0001 C CNN "Mouser Part Number"
 	1    2950 3550
 	1    0    0    -1
@@
 F 2 "Capacitor_SMD:C_0603_1608Metric" H 1550 5450 50  0001 C CNN
 F 3 "~" H 1550 5450 50  0001 C CNN
+F 4 "AVX" H 1550 5450 50  0001 C CNN "Manufacturer_Name"
+F 5 "0603YC104MAT4A" H 1550 5450 50  0001 C CNN "Manufacturer_Part_Number"
+F 6 "581-0603YC104MAT4A" H 1550 5450 50  0001 C CNN "Mouser Part Number"
 	1    1550 5450
 	1    0    0    -1
@@
 F 2 "Capacitor_SMD:C_0603_1608Metric" H 3200 5550 50  0001 C CNN
 F 3 "~" H 3200 5550 50  0001 C CNN
+F 4 "AVX" H 3200 5550 50  0001 C CNN "Manufacturer_Name"
+F 5 "0603YC104MAT4A" H 3200 5550 50  0001 C CNN "Manufacturer_Part_Number"
+F 6 "581-0603YC104MAT4A" H 3200 5550 50  0001 C CNN "Mouser Part Number"
 	1    3200 5550
 	1    0    0    -1
@@
 F 2 "Resistor_SMD:R_0603_1608Metric" V 6380 4200 50  0001 C CNN
 F 3 "~" H 6450 4200 50  0001 C CNN
-F 4 "Bourns" H 6450 4200 50  0001 C CNN "Manufacturer_Name"
-F 5 "CR0603-FX-3302ELF" H 6450 4200 50  0001 C CNN "Manufacturer_Part_Number"
-F 6 " 652-CR0603FX-3302ELF " H 6450 4200 50  0001 C CNN "Mouser Part Number"
+F 4 "Yageo" H 6450 4200 50  0001 C CNN "Manufacturer_Name"
+F 5 "RC0603FR-0733KL" H 6450 4200 50  0001 C CNN "Manufacturer_Part_Number"
+F 6 "603-RC0603FR-0733KL" H 6450 4200 50  0001 C CNN "Mouser Part Number"
 	1    6450 4200
 	0    1    1    0
@@
 F 2 "Resistor_SMD:R_0603_1608Metric" V 5980 4350 50  0001 C CNN
 F 3 "~" H 6050 4350 50  0001 C CNN
-F 4 "Bourns" H 6050 4350 50  0001 C CNN "Manufacturer_Name"
-F 5 "CR0603-FX-12R0ELF" H 6050 4350 50  0001 C CNN "Manufacturer_Part_Number"
-F 6 " 652-CR0603FX-12R0ELF " H 6050 4350 50  0001 C CNN "Mouser Part Number"
+F 4 "Yageo" H 6050 4350 50  0001 C CNN "Manufacturer_Name"
+F 5 "RC0603FR-0712RL" H 6050 4350 50  0001 C CNN "Manufacturer_Part_Number"
+F 6 " 603-RC0603FR-0712RL " H 6050 4350 50  0001 C CNN "Mouser Part Number"
 	1    6050 4350
 	-1   0    0    1
